File: compute-module.kicad_sch (KiCad schematic)
At the start: 16 parts, among them J201 DSI, SW201 SW_Push, SW202 SW_Push, U201 74154, U202 74LVC1G07SE-7

Commit message: Start placing parts on pcb.
Parts:
- SW201, SW202: footprint Button_Switch_SMD:SW_Push_1P1T_NO_6x6mm_H9.5mm -> Button_Switch_SMD:SW_SPST_B3U-1000P
Changed lines of the file:
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@@
       (effects (font (size 1.27 1.27)))
     )
-    (property "Footprint" "Button_Switch_SMD:SW_Push_1P1T_NO_6x6mm_H9.5mm" (at 46.99 176.53 0)
+    (property "Footprint" "Button_Switch_SMD:SW_SPST_B3U-1000P" (at 46.99 176.53 0)
       (effects (font (size 1.27 1.27)) hide)
     )
@@
       (effects (font (size 1.27 1.27)))
     )
-    (property "Footprint" "Button_Switch_SMD:SW_Push_1P1T_NO_6x6mm_H9.5mm" (at 46.99 166.37 0)
+    (property "Footprint" "Button_Switch_SMD:SW_SPST_B3U-1000P" (at 46.99 166.37 0)
       (effects (font (size 1.27 1.27)) hide)
     )

Commit message: Finish the draft routing.
Parts:
- renumbered C20 to C201
Changed lines of the file:
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@@
   (symbol (lib_id "Device:C_Small") (at 229.87 64.77 0) (unit 1)
     (in_bom yes) (on_board yes) (dnp no)
-    (property "Reference" "C20" (at 231.14 63.5 0)
+    (property "Reference" "C201" (at 231.14 63.5 0)
       (effects (font (size 1.27 1.27)) (justify left))
     )
@@
     (instances
       (project "main-board"
-        (path "/5ad67b7d-c56f-4b00-8953-cc84f90f9708/72ca2a69-64d2-4325-ac9e-ca976eb5a207"
-          (reference "C20") (unit 1)
-        )
         (path "/5ad67b7d-c56f-4b00-8953-cc84f90f9708/d4025ecd-c2b7-426a-90ae-23d9d1364d9e"
           (reference "C201") (unit 1)
