File: compute-module.kicad_sch (KiCad schematic)
At the start: 16 parts, among them J201 DSI, SW201 SW_Push, SW202 SW_Push, U201 74154, U202 74LVC1G07SE-7

Commit message: Update MPNs.
Parts:
- C201: MPN RM EMK105 B7104KV-F -> C0603C104K4RAC7081
- SW201, SW202: MPN TS04-66-65-BK-100-SMT -> B3U-1000P
Changed lines of the file:
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@@
       (effects (font (size 1.27 1.27)) hide)
     )
-    (property "MPN" "RM EMK105 B7104KV-F" (at 229.87 64.77 0)
+    (property "MPN" "C0603C104K4RAC7081" (at 229.87 64.77 0)
       (effects (font (size 1.27 1.27)) hide)
     )
@@
       (effects (font (size 1.27 1.27)) hide)
     )
-    (property "MPN" "TS04-66-65-BK-100-SMT" (at 46.99 181.61 0)
+    (property "MPN" "B3U-1000P" (at 46.99 181.61 0)
       (effects (font (size 1.27 1.27)) hide)
     )
@@
       (effects (font (size 1.27 1.27)) hide)
     )
-    (property "MPN" "TS04-66-65-BK-100-SMT" (at 46.99 171.45 0)
-      (effects (font (size 1.27 1.27)) hide)
-    )
+    (property "MPN" "B3U-1000P" (at 46.99 171.45 0)
+      (effects (font (size 1.27 1.27)) hide)
+    )

Commit message: Add MPNs for CM4 and motor drivers.
Parts:
- Module201: MPN (none) -> 2x DF40C-100DS-0.4V(51)
Changed lines of the file:
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@@
+      (effects (font (size 1.27 1.27)) hide)
+    )
+    (property "MPN" "2x DF40C-100DS-0.4V(51)" (at 13.97 86.36 0)
       (effects (font (size 1.27 1.27)) hide)
     )
@@
       (effects (font (size 1.27 1.27)) hide)
     )
+    (property "MPN" "2x DF40C-100DS-0.4V(51)" (at 67.31 81.28 0)
+      (effects (font (size 1.27 1.27)) hide)
+    )

Commit message: Fix the issues found during testing in schematics.
Parts:
- removed R202, R203: 2.2K, Resistor_SMD:R_0603_1608Metric, symbol Device:R_Small_US
Connections:
- net GPIO3 is gone; now on net ~{SHUT_DOWN}: Module201.56 (GPIO3)
- net GND: now also J201.14 (Pin_14), J201.15 (Pin_15), Module201.194 (DSI1_D3_N), Module201.196 (DSI1_D3_P)
- net ~{POWER_OFF}: now also Module201.54 (GPIO4); no longer Module201.24 (GPIO26)
- net ~{SHUT_DOWN}: no longer Module201.54 (GPIO4)
- net DSI1_D2_N: now reaches J201.11 (Pin_11)
- net DSI1_D2_N: now also Module201.193 (DSI1_D2_N)
- net DSI1_D2_P: now reaches J201.12 (Pin_12)
- net DSI1_D2_P: now also Module201.195 (DSI1_D2_P)
- net DSI1_D0_N: now reaches Module201.175 (DSI1_D0_N)
- net DSI1_D0_N: now also J201.2 (Pin_2)
- net DSI1_D0_P: now reaches Module201.177 (DSI1_D0_P)
- net DSI1_D0_P: now also J201.3 (Pin_3)
- net DSI1_D1_N: now reaches Module201.181 (DSI1_D1_N)
- net DSI1_D1_N: now also J201.5 (Pin_5)
- net DSI1_D1_P: now reaches Module201.183 (DSI1_D1_P)
- net DSI1_D1_P: now also J201.6 (Pin_6)
- net DSI1_C_N: now reaches Module201.187 (DSI1_C_N)
- net DSI1_C_N: now also J201.8 (Pin_8)
- net DSI1_C_P: now reaches Module201.189 (DSI1_C_P)
- net DSI1_C_P: now also J201.9 (Pin_9)
- net SCL0: now reaches Module201.80 (SCL0)
- net SCL0: now also J201.20 (Pin_20)
- net SDA0: now reaches Module201.82 (SDA0)
- net SDA0: now also J201.21 (Pin_21)
- net DSI0_C_N: no longer names the net of Module201.169 (DSI0_C_N)
- net DSI0_C_N: no longer J201.8 (Pin_8)
- net DSI0_C_P: no longer names the net of Module201.171 (DSI0_C_P)
- net DSI0_C_P: no longer J201.9 (Pin_9)
- net DSI0_D0_N: no longer names the net of Module201.157 (DSI0_D0_N)
- net DSI0_D0_N: no longer J201.2 (Pin_2)
- net DSI0_D0_P: no longer names the net of Module201.159 (DSI0_D0_P)
- net DSI0_D0_P: no longer J201.3 (Pin_3)
- net DSI0_D1_N: no longer names the net of Module201.163 (DSI0_D1_N)
- net DSI0_D1_N: no longer J201.5 (Pin_5)
- net DSI0_D1_P: no longer names the net of Module201.165 (DSI0_D1_P)
- net DSI0_D1_P: no longer J201.6 (Pin_6)
- net ID_SC: no longer names the net of Module201.35 (ID_SC)
- net ID_SC: no longer J201.20 (Pin_20)
- net ID_SD: no longer names the net of Module201.36 (ID_SD)
- net ID_SD: no longer J201.21 (Pin_21)
- new net GPIO26: Module201.24 (GPIO26)
- no-connect marks 111 -> 103
Other:
- moved on the sheet: Module201B

Commit message: Change on-board LEDs to vertical diffuse.
Parts:
- D201: MPN SML-A12U8TT86Q -> B1911USD-20D000114U1930
- D202: MPN SML-A12M8TT86N -> B1911PG--20D000514U1930
Changed lines of the file:
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@@
       (effects (font (size 1.27 1.27)) hide)
     )
-    (property "MPN" "SML-A12U8TT86Q" (at 105.41 168.91 0)
+    (property "MPN" "B1911USD-20D000114U1930" (at 105.41 168.91 0)
       (effects (font (size 1.27 1.27)) hide)
     )
@@
       (effects (font (size 1.27 1.27)) hide)
     )
-    (property "MPN" "SML-A12M8TT86N" (at 130.81 168.91 0)
-      (effects (font (size 1.27 1.27)) hide)
-    )
+    (property "MPN" "B1911PG--20D000514U1930" (at 130.81 168.91 0)
+      (effects (font (size 1.27 1.27)) hide)
+    )
