File: power.kicad_sch (KiCad schematic)
At the start: 40 parts, among them J1 Conn_01x02, Q1 BSC014N04LS, SW3 SW_Push, U3 AP64501SP-13, U4 LTC2955CTS8-1, U5 LTC4231-2, U6 PAC1954

Commit message: Add RP2040
Parts:
- C7, C8: value 100n -> 100nF
Changed lines of the file:
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@@
       (effects (font (size 1.27 1.27)) (justify left))
     )
-    (property "Value" "100n" (at 111.76 124.46 0)
+    (property "Value" "100nF" (at 111.76 124.46 0)
       (effects (font (size 1.27 1.27)) (justify left))
     )
@@
       (effects (font (size 1.27 1.27)) (justify left))
     )
-    (property "Value" "100n" (at 123.19 147.32 0)
-      (effects (font (size 1.27 1.27)) (justify left))
-    )
+    (property "Value" "100nF" (at 123.19 147.32 0)
+      (effects (font (size 1.27 1.27)) (justify left))
+    )

Commit message: Finish connecting everything in sch.
Parts:
- removed J1: Conn_01x02, symbol Connector_Generic:Conn_01x02
Connections:
- net -BATT renamed GND
Changed lines of the file:
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@@
   (junction (at 54.61 132.08) (diameter 0) (color 0 0 0 0)
   )
-  (junction (at 60.96 71.12) (diameter 0) (color 0 0 0 0)
-  )
   (junction (at 41.91 43.18) (diameter 0) (color 0 0 0 0)
   )
@@
     (stroke (width 0) (type solid))
   )
-  (wire (pts (xy 59.69 71.12) (xy 60.96 71.12))
-    (stroke (width 0) (type default))
-  )
   (wire (pts (xy 213.36 26.67) (xy 213.36 27.94))
     (stroke (width 0) (type default))
@@
     (stroke (width 0) (type solid))
   )
-  (wire (pts (xy 59.69 68.58) (xy 62.23 68.58))
-    (stroke (width 0) (type default))
-  )
   (wire (pts (xy 167.64 125.73) (xy 177.8 125.73))
     (stroke (width 0) (type solid))
@@
     (stroke (width 0) (type default))
   )
-  (wire (pts (xy 60.96 71.12) (xy 62.23 71.12))
-    (stroke (width 0) (type default))
-  )
   (wire (pts (xy 52.07 40.64) (xy 54.61 40.64))
     (stroke (width 0) (type default))
@@
   (wire (pts (xy 86.36 139.7) (xy 86.36 138.43))
     (stroke (width 0) (type solid))
-  )
-  (wire (pts (xy 60.96 71.12) (xy 60.96 72.39))
-    (stroke (width 0) (type default))
   )
   (wire (pts (xy 187.96 124.46) (xy 187.96 125.73))
@@
         (path "/e63e39d7-6ac0-4ffd-8aa3-1841a4541b55/00000000-0000-0000-0000-00005d31f999"
           (reference "#PWR0120") (unit 1)
-        )
-      )
-    )
-  )
-  (symbol (lib_id "Connector_Generic:Conn_01x02") (at 67.31 68.58 0) (unit 1)
-    (in_bom yes) (on_board yes) (dnp no) (fields_autoplaced)
-    (property "Reference" "J1" (at 69.85 69.215 0)
-      (effects (font (size 1.27 1.27)) (justify left))
-    )
-    (property "Value" "Conn_01x02" (at 69.85 71.755 0)
-      (effects (font (size 1.27 1.27)) (justify left))
-    )
-    (property "Footprint" "" (at 67.31 68.58 0)
-      (effects (font (size 1.27 1.27)) hide)
-    )
-    (property "Datasheet" "~" (at 67.31 68.58 0)
-      (effects (font (size 1.27 1.27)) hide)
-    )
-    (pin "1")
-    (pin "2")
-    (instances
-      (project "main-board"
-        (path "/5ad67b7d-c56f-4b00-8953-cc84f90f9708/a004841b-bac3-4d41-b697-5d2e29fa9f3a"
-          (reference "J1") (unit 1)
         )
       )
@@
     )
   )
-  (symbol (lib_id "power:-BATT") (at 59.69 71.12 90) (unit 1)
-    (in_bom yes) (on_board yes) (dnp no)
-    (property "Reference" "#PWR023" (at 63.5 71.12 0)
-      (effects (font (size 1.27 1.27)) hide)
-    )
-    (property "Value" "-BATT" (at 57.15 71.12 90)
-      (effects (font (size 1.27 1.27)) (justify left))
-    )
-    (property "Footprint" "" (at 59.69 71.12 0)
-      (effects (font (size 1.27 1.27)) hide)
-    )
-    (property "Datasheet" "" (at 59.69 71.12 0)
-      (effects (font (size 1.27 1.27)) hide)
-    )
-    (pin "1")
-    (instances
-      (project "main-board"
-        (path "/5ad67b7d-c56f-4b00-8953-cc84f90f9708/a004841b-bac3-4d41-b697-5d2e29fa9f3a"
-          (reference "#PWR023") (unit 1)
-        )
-      )
-    )
-  )
   (symbol (lib_id "Device:R_Small_US") (at 36.83 31.75 0) (unit 1)
     (in_bom yes) (on_board yes) (dnp no)
@@
         (path "/e63e39d7-6ac0-4ffd-8aa3-1841a4541b55/00000000-0000-0000-0000-00005d31f999"
           (reference "R28") (unit 1)
-        )
-      )
-    )
-  )
-  (symbol (lib_id "power:+BATT") (at 59.69 68.58 90) (unit 1)
-    (in_bom yes) (on_board yes) (dnp no) (fields_autoplaced)
-    (property "Reference" "#PWR026" (at 63.5 68.58 0)
-      (effects (font (size 1.27 1.27)) hide)
-    )
-    (property "Value" "+BATT" (at 55.88 69.215 90)
-      (effects (font (size 1.27 1.27)) (justify left))
-    )
-    (property "Footprint" "" (at 59.69 68.58 0)
-      (effects (font (size 1.27 1.27)) hide)
-    )
-    (property "Datasheet" "" (at 59.69 68.58 0)
-      (effects (font (size 1.27 1.27)) hide)
-    )
-    (pin "1")
-    (instances
-      (project "main-board"
-        (path "/5ad67b7d-c56f-4b00-8953-cc84f90f9708/a004841b-bac3-4d41-b697-5d2e29fa9f3a"
-          (reference "#PWR026") (unit 1)
         )
       )
@@
         )
       )
-    )
-  )
-  (symbol (lib_name "GND_1") (lib_id "power:GND") (at 60.96 72.39 0) (unit 1)
-    (in_bom yes) (on_board yes) (dnp no)
-    (property "Reference" "#PWR027" (at 60.96 78.74 0)
-      (effects (font (size 1.27 1.27)) hide)
-    )
-    (property "Value" "GND" (at 60.96 77.47 0)
-      (effects (font (size 1.27 1.27)))
-    )
-    (property "Footprint" "" (at 60.96 72.39 0)
-      (effects (font (size 1.27 1.27)) hide)
-    )
-    (property "Datasheet" "" (at 60.96 72.39 0)
-      (effects (font (size 1.27 1.27)) hide)
-    )
-    (pin "1")
-    (instances
-      (project "main-board"
-        (path "/5ad67b7d-c56f-4b00-8953-cc84f90f9708/a004841b-bac3-4d41-b697-5d2e29fa9f3a"
-          (reference "#PWR027") (unit 1)
-        )
-      )

Commit message: Fix sch errors and warnings.
Parts:
- C16: symbol Device:CP -> Device:C_Polarized_Small
- L1: value SRN6045TA-3R3Y -> 3.3µH; symbol pspice:INDUCTOR -> Device:L; Field4 Farnell -> (none); Field5 2616889 -> (none); Field6 SRN6045TA-3R3Y -> (none); Field7 Bourns -> (none); MPN (none) -> SRN6045TA-3R3Y; Part Description 3.3µH Semi-Shielded Wirewound Inductor 7.8A 21mOhm Nonstand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 -> (none)
Connections:
- net SENSE_MIKONA- renamed SENSE_MIKONA
- no-connect marks 0 -> 4
Other:
- moved on the sheet: R19, R20, U6

Commit message: Assign some of the footprints and MPNs.
Parts:
- C1, C2, C3, C4, C5, C6: Field4 Digikey -> (none); Field5 490-10505-1-ND -> (none); Field6 GRM21BC8YA106KE11L -> (none); Field7 Murata -> (none); MPN (none) -> GRM21BC8YA106KE11L; Part Description 10uF 10% or 20% 35V Ceramic Capacitor X6S 0805 (2012 Metric) -> (none)
- C10: Field4 Digikey -> (none); Field5 490-16429-1-ND -> (none); Field6 GCM155R71H122KA37D -> (none); Field7 Murata -> (none); MPN (none) -> GCM155R71H122KA37D; Part Description 1200pF 10% 10V Ceramic Capacitor X5R 0402 (1005 Metric) -> (none)
- C12, C13, C14, C15: Field4 Digikey -> (none); Field5 490-14381-1-ND -> (none); Field6 GRM21BR71A106KA73L -> (none); Field7 Murata -> (none); Field8 111893011 -> (none); MPN (none) -> GRM21BR71A106KA73L; Part Description 10uF 10% 10V Ceramic Capacitor X7R 0805 (2012 Metric) -> (none)
- C16: Field4 Mouser -> (none); Field5 667-EEF-CX0J101R -> (none); Part Description Capacitor, SP-Cap, 100u, 6.3V, 15mR ESR -> (none)
- C7, C8: Field4 Farnell -> (none); Field5 2611911 -> (none); Field6 RM EMK105 B7104KV-F -> (none); Field7 TAIYO YUDEN EUROPE GMBH -> (none); Field8 110091611 -> (none); MPN (none) -> RM EMK105 B7104KV-F; Part Description 0.1uF 10% 16V Ceramic Capacitor X7R 0402 (1005 Metric) -> (none)
- C9: footprint (none) -> Capacitor_SMD:C_0402_1005Metric
- Q1: AVAILABILITY Good -> (none); DESCRIPTION MOSFET Transistor, N Channel, 100 A, 40 V, 0.0012 ohm, 10 V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 -> (none); MF Infineon Technologies -> (none); MP BSC014N04LSIATMA1 -> (none); MPN (none) -> BSC014N04LSIATMA1; PACKAGE PowerTDFN-8 Infineon -> (none); PRICE 1.90 USD -> (none)
- R10: Field4 Farnell -> (none); Field5 9239278 -> (none); Field6 RK73G1ETQTP2201D -> (none); Field7 KOA EUROPE GMBH -> (none); Field8 120889581 -> (none); MPN (none) -> RK73G1ETQTP2201D; Part Description Resistor 2.2K M1005 1% 63mW -> (none)
- R11, R12, R13, R14, R15, R18, R19, R20: footprint (none) -> Resistor_SMD:R_0402_1005Metric
- R7: Field4 Farnell -> (none); Field5 9238999 -> (none); Field6 RC0402FR-0710RL -> (none); Field7 Yageo -> (none); Field8 URES00256 -> (none); MPN (none) -> RC0402FR-0710RL; Part Description Resistor 10R M1005 1% 63mW -> (none)
- R8: Field4 Farnell -> (none); Field5 2331485 -> (none); Field6 RK73H1ETTP2002F -> (none); Field7 KOA EUROPE GMBH -> (none); MPN (none) -> RK73H1ETTP2002F; Part Description Resistor 20K M1005 1% 63mW -> (none)
- R9: Field4 Farnell -> (none); Field5 9239367 -> (none); Field6 MCR01MZPF1202 -> (none); Field7 Rohm -> (none); MPN (none) -> MCR01MZPF1202; Part Description Resistor 12K M1005 1% 63mW -> (none)
- SW3: footprint (none) -> Button_Switch_THT:SW_Tactile_SPST_Angled_PTS645Vx58-2LFS; MPN (none) -> 1825027-8
- U3: Field4 Digikey -> (none); Field5 31-AP64501SP-13CT-ND -> (none); Field6 AP64501SP-13 -> (none); Field7 Diodes -> (none); MPN (none) -> AP64501SP-13; Part Description Buck Switching Regulator IC Positive Adjustable 0.8V 1 Outp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 -> (none)
- U4: MANUFACTURER_PART_NUMBER ltc2955cts81#pbf -> (none); VENDOR Linear Technology -> (none)
- U5: MANUFACTURER Linear Technology -> (none); PARTREV A -> (none); STANDARD IPC-7351B -> (none)

Commit message: Import the previous main board to match the overall shape, and re-annotate the schematic.
Parts:
- C301: renamed from C17; footprint (none) -> Capacitor_SMD:C_0805_2012Metric
- C302: renamed from C18; footprint (none) -> Capacitor_SMD:C_0603_1608Metric
- C303: renamed from C9; footprint Capacitor_SMD:C_0402_1005Metric -> Capacitor_SMD:C_0603_1608Metric; MPN (none) -> RM EMK105 B7104KV-F
- C304: renamed from C19; footprint (none) -> Capacitor_SMD:C_0603_1608Metric
- C309: renamed from C7; footprint Capacitor_SMD:C_0402_1005Metric -> Capacitor_SMD:C_0603_1608Metric
- C317: renamed from C8; footprint Capacitor_SMD:C_0402_1005Metric -> Capacitor_SMD:C_0603_1608Metric
- C318: renamed from C10; footprint Capacitor_SMD:C_0402_1005Metric -> Capacitor_SMD:C_0603_1608Metric
- R301: renamed from R16; footprint (none) -> Resistor_SMD:R_2512_6332Metric
- R302: renamed from R17; footprint (none) -> Resistor_SMD:R_2512_6332Metric
- R303: renamed from R11; footprint Resistor_SMD:R_0402_1005Metric -> Resistor_SMD:R_0603_1608Metric; MPN (none) -> RC0603FR-101KL
- R304: renamed from R12; footprint Resistor_SMD:R_0402_1005Metric -> Resistor_SMD:R_0603_1608Metric
- R305: renamed from R20; footprint Resistor_SMD:R_0402_1005Metric -> Resistor_SMD:R_0603_1608Metric; MPN (none) -> RC0603FR-101KL
- R306: renamed from R13; footprint Resistor_SMD:R_0402_1005Metric -> Resistor_SMD:R_0603_1608Metric
- R307: renamed from R14; footprint Resistor_SMD:R_0402_1005Metric -> Resistor_SMD:R_0603_1608Metric
- R308: renamed from R19; footprint Resistor_SMD:R_0402_1005Metric -> Resistor_SMD:R_0603_1608Metric; MPN (none) -> RC0603FR-101KL
- R309: renamed from R15; footprint Resistor_SMD:R_0402_1005Metric -> Resistor_SMD:R_0603_1608Metric
- R310: renamed from R7; value 10R -> 10; footprint Resistor_SMD:R_0402_1005Metric -> Resistor_SMD:R_0603_1608Metric
- R311: renamed from R18; footprint Resistor_SMD:R_0402_1005Metric -> Resistor_SMD:R_0603_1608Metric; MPN (none) -> RC0603FR-101KL
- R312: renamed from R9; footprint Resistor_SMD:R_0402_1005Metric -> Resistor_SMD:R_0603_1608Metric
- R313: renamed from R8; footprint Resistor_SMD:R_0402_1005Metric -> Resistor_SMD:R_0603_1608Metric
- R314: renamed from R10; footprint Resistor_SMD:R_0402_1005Metric -> Resistor_SMD:R_0603_1608Metric
- renumbered C12 to C305, C13 to C306, C14 to C307, C15 to C308, C16 to C310, C1 to C311, C2 to C312, C3 to C313, C4 to C314, C5 to C315, C6 to C316, L1 to L301, Q1 to Q301, SW3 to SW301, U4 to U301, U6 to U302, U5 to U303, U3 to U304

Commit message: Finish the draft routing.
Parts:
- added D202: LED Green, LED_SMD:LED_0603_1608Metric, symbol Device:LED
- added R206: 1K, Resistor_SMD:R_0603_1608Metric, symbol Device:R_Small_US
- R311: value 1K -> 2mΩ
Connections:
- net +24V: now also U302.13 (SENSE2+), R206.1; no longer U302.8 (SENSE3+)
- net +5V: now also C305.1, C306.1, C307.1, C308.1, C310.1, L301.2, R312.1; no longer R311.1, U302.14 (SENSE2-)
- net +BATT: now also R311.2; no longer C311.1, C312.1, C313.1, C314.1, C315.1, C316.1, U304.2 (VIN)
- net GND: now also D202.1 (K)
- net PWR_STATUS: no longer names the net of U303.9 (STATUS)
- net PWR_STATUS: now also D202.2 (A), R206.2
- removed net SENSE_5v+: C305.1, C306.1, C307.1, C308.1, C310.1, L301.2, R311.2, R312.1, U302.13 (SENSE2+)
- net SENSE_MIKONA: no longer names the net of U302.7 (SENSE3-)
- new net SENSE_5v-: C311.1, C312.1, C313.1, C314.1, C315.1, C316.1, R311.1, U302.14 (SENSE2-), U304.2 (VIN)
- no-connect marks 4 -> 6
Other:
- moved on the sheet: C305, C306, C307, C308, C309, C310, C311, C312, C313, C314, C315, C316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

Commit message: Improve routings,
Parts:
- U304: footprint Package_SO:SOIC-8-1EP_3.9x4.9mm_P1.27mm_EP2.95x4.9mm_Mask2.71x3.4mm_ThermalVias -> Package_SO:SOIC-8-1EP_3.9x4.9mm_P1.27mm_EP2.62x3.51mm
Changed lines of the file:
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@@
       (effects (font (size 1.27 1.27)))
     )
-    (property "Footprint" "Package_SO:SOIC-8-1EP_3.9x4.9mm_P1.27mm_EP2.95x4.9mm_Mask2.71x3.4mm_ThermalVias" (at 156.21 132.08 0)
+    (property "Footprint" "Package_SO:SOIC-8-1EP_3.9x4.9mm_P1.27mm_EP2.62x3.51mm" (at 156.21 132.08 0)
       (effects (font (size 1.27 1.27)) hide)
     )

Commit message: Improve routings.
Parts:
- R311: footprint Resistor_SMD:R_0603_1608Metric -> Resistor_SMD:R_2512_6332Metric; MPN RC0603FR-101KL -> (none)
Changed lines of the file:
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@@
       (effects (font (size 1.27 1.27)) (justify left))
     )
-    (property "Footprint" "Resistor_SMD:R_0603_1608Metric" (at 60.96 132.08 0)
+    (property "Footprint" "Resistor_SMD:R_2512_6332Metric" (at 60.96 132.08 0)
       (effects (font (size 1.27 1.27)) hide)
     )
@@
       (effects (font (size 1.27 1.27)) hide)
     )
-    (property "MPN" "RC0603FR-101KL" (at 60.96 132.08 0)
+    (property "MPN" "" (at 60.96 132.08 0)
       (effects (font (size 1.27 1.27)) hide)
     )
