File: power.kicad_sch (KiCad schematic)
At the start: 41 parts, among them Q301 BSC014N04LS, SW301 SW_Push, U301 LTC2955CTS8-1, U302 PAC1954, U303 LTC4231-2, U304 AP64501SP-13

Commit message: Update MPNs.
Parts:
- C301: MPN (none) -> C0805C103K1RAC7025
- C302: MPN (none) -> GRM188R71E474KA12J
- C303, C309, C317: MPN RM EMK105 B7104KV-F -> C0603C104K4RAC7081
- C304: MPN (none) -> GCM188R71E184KA55D
- C310: MPN (none) -> T491D107K010AT
- C318: MPN GCM155R71H122KA37D -> C0603C122K5RAC7867
- R301: MPN (none) -> EBWM2512F1L00S9
- R302, R311: MPN (none) -> PEWF2512F2L00Q9
- R304: MPN (none) -> RC0603DR-071ML
- R306: MPN (none) -> RT0603DRE075K6L
- R307: MPN (none) -> RT0603DRE0740K2L
- R309: MPN (none) -> RT0603DRE0724KL
- R310: MPN RC0402FR-0710RL -> RC0603FR-1010RL
- R312: MPN MCR01MZPF1202 -> RC0603FR-1312KL
- R313: MPN RK73H1ETTP2002F -> RC0603FR-0720KL
- R314: MPN RK73G1ETQTP2201D -> RC0603FR-132K2L
- U301: MPN (none) -> LTC2955CTS8-1#TRMPBF
- U302: MPN (none) -> PAC1954T-E/4MX
- U303: MPN (none) -> LTC4231CMS-2#PBF
Changed lines of the file:
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@@
       (effects (font (size 1.27 1.27)) hide)
     )
-    (property "MPN" "MCR01MZPF1202" (at 187.96 129.54 0)
+    (property "MPN" "RC0603FR-1312KL" (at 187.96 129.54 0)
       (effects (font (size 1.27 1.27)) hide)
     )
@@
     )
     (property "Datasheet" "~" (at 118.11 53.34 0)
+      (effects (font (size 1.27 1.27)) hide)
+    )
+    (property "MPN" "RT0603DRE075K6L" (at 118.11 53.34 0)
       (effects (font (size 1.27 1.27)) hide)
     )
@@
       (effects (font (size 1.27 1.27)) hide)
     )
+    (property "MPN" "PEWF2512F2L00Q9" (at 167.64 29.21 0)
+      (effects (font (size 1.27 1.27)) hide)
+    )
     (pin "1")
     (pin "2")
@@
       (effects (font (size 1.27 1.27)) hide)
     )
+    (property "MPN" "T491D107K010AT" (at 236.22 123.19 0)
+      (effects (font (size 1.27 1.27)) hide)
+    )
     (pin "1")
     (pin "2")
@@
       (effects (font (size 1.27 1.27)) hide)
     )
-    (property "MPN" "RM EMK105 B7104KV-F" (at 143.51 123.19 0)
+    (property "MPN" "C0603C104K4RAC7081" (at 143.51 123.19 0)
       (effects (font (size 1.27 1.27)) hide)
     )
@@
     )
     (property "Datasheet" "~" (at 125.73 29.21 0)
+      (effects (font (size 1.27 1.27)) hide)
+    )
+    (property "MPN" "EBWM2512F1L00S9" (at 125.73 29.21 0)
       (effects (font (size 1.27 1.27)) hide)
     )
@@
       (effects (font (size 1.27 1.27)) hide)
     )
-    (property "MPN" "RM EMK105 B7104KV-F" (at 247.65 46.99 0)
+    (property "MPN" "C0603C104K4RAC7081" (at 247.65 46.99 0)
       (effects (font (size 1.27 1.27)) hide)
     )
@@
     )
     (property "Datasheet" "~" (at 118.11 48.26 0)
+      (effects (font (size 1.27 1.27)) hide)
+    )
+    (property "MPN" "RC0603DR-071ML" (at 118.11 48.26 0)
       (effects (font (size 1.27 1.27)) hide)
     )
@@
       (effects (font (size 1.27 1.27)) hide)
     )
+    (property "MPN" "LTC2955CTS8-1#TRMPBF" (at 54.61 35.56 0)
+      (effects (font (size 1.27 1.27)) hide)
+    )
     (pin "1")
     (pin "3")
@@
       (effects (font (size 1.27 1.27)) hide)
     )
-    (property "MPN" "GCM155R71H122KA37D" (at 173.99 149.86 0)
+    (property "MPN" "C0603C122K5RAC7867" (at 173.99 149.86 0)
       (effects (font (size 1.27 1.27)) hide)
     )
@@
       (effects (font (size 1.27 1.27)) hide)
     )
-    (property "MPN" "RC0402FR-0710RL" (at 148.59 118.11 0)
+    (property "MPN" "RC0603FR-1010RL" (at 148.59 118.11 0)
       (effects (font (size 1.27 1.27)) hide)
     )
@@
       (effects (font (size 1.27 1.27)) hide)
     )
-    (property "MPN" "RM EMK105 B7104KV-F" (at 147.32 146.05 0)
+    (property "MPN" "C0603C104K4RAC7081" (at 147.32 146.05 0)
       (effects (font (size 1.27 1.27)) hide)
     )
@@
       (effects (font (size 1.27 1.27)) hide)
     )
-    (property "MPN" "RK73H1ETTP2002F" (at 173.99 142.24 0)
+    (property "MPN" "RC0603FR-0720KL" (at 173.99 142.24 0)
       (effects (font (size 1.27 1.27)) hide)
     )
@@
       (effects (font (size 1.27 1.27)) hide)
     )
-    (property "MPN" "" (at 60.96 132.08 0)
+    (property "MPN" "PEWF2512F2L00Q9" (at 60.96 132.08 0)
       (effects (font (size 1.27 1.27)) hide)
     )
@@
     )
     (property "Datasheet" "~" (at 160.02 66.04 0)
+      (effects (font (size 1.27 1.27)) hide)
+    )
+    (property "MPN" "GCM188R71E184KA55D" (at 160.02 66.04 0)
       (effects (font (size 1.27 1.27)) hide)
     )
@@
       (effects (font (size 1.27 1.27)) hide)
     )
-    (property "MPN" "RK73G1ETQTP2201D         " (at 187.96 146.05 0)
+    (property "MPN" "RC0603FR-132K2L" (at 187.96 146.05 0)
       (effects (font (size 1.27 1.27)) hide)
     )
@@
       (effects (font (size 1.27 1.27)) hide)
     )
+    (property "MPN" "RT0603DRE0724KL" (at 118.11 63.5 0)
+      (effects (font (size 1.27 1.27)) hide)
+    )
     (pin "1")
     (pin "2")
@@
     )
     (property "Datasheet" "~" (at 88.9 45.72 0)
+      (effects (font (size 1.27 1.27)) hide)
+    )
+    (property "MPN" "GRM188R71E474KA12J" (at 88.9 45.72 0)
       (effects (font (size 1.27 1.27)) hide)
     )
@@
       (effects (font (size 1.27 1.27)) hide)
     )
+    (property "MPN" "C0805C103K1RAC7025" (at 36.83 39.37 0)
+      (effects (font (size 1.27 1.27)) hide)
+    )
     (pin "1")
     (pin "2")
@@
       (effects (font (size 1.27 1.27)) hide)
     )
+    (property "MPN" "RT0603DRE0740K2L" (at 118.11 58.42 0)
+      (effects (font (size 1.27 1.27)) hide)
+    )
     (pin "1")
     (pin "2")
@@
     )
     (property "Datasheet" "https://ww1.microchip.com/downloads/en/DeviceDoc/PAC195X-Data-Sheet-20006539.pdf" (at 214.63 83.82 0)
+      (effects (font (size 1.27 1.27)) hide)
+    )
+    (property "MPN" "PAC1954T-E/4MX" (at 214.63 48.26 0)
       (effects (font (size 1.27 1.27)) hide)
     )
@@
       (effects (font (size 1.27 1.27)) hide)
     )
+    (property "MPN" "LTC4231CMS-2#PBF" (at 139.7 55.88 0)
+      (effects (font (size 1.27 1.27)) hide)
+    )

Commit message: Fix the issues found during testing in schematics.
Parts:
- removed D202: LED Green, LED_SMD:LED_0603_1608Metric, symbol Device:LED
- added R206 (x2), R316: 1K, Resistor_SMD:R_0603_1608Metric, symbol Device:R_Small_US
- SW301: value SW_Push -> 228ADS2; footprint Button_Switch_THT:SW_Tactile_SPST_Angled_PTS645Vx58-2LFS -> 228ADS2:228ADS2; symbol Switch:SW_Push -> 228ADS2:228ADS2; MPN 1825027-8 -> 228ADS2AAWFCMBA
Connections:
- net +3.3V: now also R316.2
- net +5V: now also R206.2
- net GND: now also SW301.2, R206.2
- net ~{PWR_KILL}: now also R316.1
- net at U301.5 (~{PB}): now also SW301.3, SW301.4; no longer SW301.2
- new net: R206.1, R206.1, SW301.L2
- new net LED_SWITCH: SW301.L1
Other:
- moved on the sheet: C301, R206, R303

Commit message: Applied the fixes to the PCB as well.
Other:
- moved on the sheet: R206
Changed lines of the file:
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@@
     (stroke (width 0) (type solid))
-  )
-  (wire (pts (xy 166.37 33.02) (xy 175.26 33.02))
-    (stroke (width 0) (type default))
   )
   (wire (pts (xy 165.1 118.11) (xy 165.1 129.54))
@@
     (stroke (width 0) (type default))
   )
-  (wire (pts (xy 166.37 54.61) (xy 166.37 44.45))
+  (wire (pts (xy 175.26 54.61) (xy 175.26 44.45))
     (stroke (width 0) (type default))
   )
@@
     (stroke (width 0) (type default))
   )
-  (wire (pts (xy 175.26 33.02) (xy 175.26 29.21))
-    (stroke (width 0) (type default))
-  )
   (wire (pts (xy 33.02 41.91) (xy 34.29 41.91))
     (stroke (width 0) (type default))
@@
     (stroke (width 0) (type default))
   )
-  (wire (pts (xy 166.37 33.02) (xy 166.37 39.37))
+  (wire (pts (xy 175.26 29.21) (xy 175.26 39.37))
     (stroke (width 0) (type default))
   )
@@
     (stroke (width 0) (type default))
   )
-  (wire (pts (xy 157.48 54.61) (xy 166.37 54.61))
+  (wire (pts (xy 157.48 54.61) (xy 175.26 54.61))
     (stroke (width 0) (type default))
   )
@@
     )
   )
-  (symbol (lib_id "Device:R_Small_US") (at 166.37 41.91 0) (unit 1)
-    (in_bom yes) (on_board yes) (dnp no)
-    (property "Reference" "R206" (at 168.148 40.7416 0)
-      (effects (font (size 1.27 1.27)) (justify left))
-    )
-    (property "Value" "1K" (at 168.148 43.053 0)
-      (effects (font (size 1.27 1.27)) (justify left))
-    )
-    (property "Footprint" "Resistor_SMD:R_0603_1608Metric" (at 166.37 41.91 0)
-      (effects (font (size 1.27 1.27)) hide)
-    )
-    (property "Datasheet" "~" (at 166.37 41.91 0)
-      (effects (font (size 1.27 1.27)) hide)
-    )
-    (property "MPN" "RC0603FR-101KL" (at 166.37 41.91 0)
-      (effects (font (size 1.27 1.27)) hide)
-    )
+  (symbol (lib_id "Device:R_Small_US") (at 175.26 41.91 0) (unit 1)
+    (in_bom yes) (on_board yes) (dnp no)
+    (property "Reference" "R206" (at 168.91 40.64 0)
+      (effects (font (size 1.27 1.27)) (justify left))
+    )
+    (property "Value" "1K" (at 171.45 43.18 0)
+      (effects (font (size 1.27 1.27)) (justify left))
+    )
+    (property "Footprint" "Resistor_SMD:R_0603_1608Metric" (at 175.26 41.91 0)
+      (effects (font (size 1.27 1.27)) hide)
+    )
+    (property "Datasheet" "~" (at 175.26 41.91 0)
+      (effects (font (size 1.27 1.27)) hide)
+    )
+    (property "MPN" "RC0603FR-101KL" (at 175.26 41.91 0)
+      (effects (font (size 1.27 1.27)) hide)
+    )

Commit message: More refinements to the PCB.
Parts:
- added TP301: 24V, TestPoint:TestPoint_Pad_D2.0mm, symbol Connector:TestPoint
- added TP302: 5V, TestPoint:TestPoint_Pad_D2.0mm, symbol Connector:TestPoint
- added TP303: 3.3V, TestPoint:TestPoint_Pad_D2.0mm, symbol Connector:TestPoint
- added TP304: GND, TestPoint:TestPoint_Pad_D2.0mm, symbol Connector:TestPoint
Connections:
- net +24V: now also TP301.1
- net +3.3V: now also TP303.1
- net +5V: now also TP302.1
- net GND: now also TP304.1
Other:
- note added: "Test points"
Changed lines of the file:
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@@
+    (stroke (width 0) (type default))
+  )
+  (wire (pts (xy 58.42 81.28) (xy 58.42 82.55))
     (stroke (width 0) (type default))
   )
@@
     (stroke (width 0) (type solid))
   )
+  (wire (pts (xy 33.02 81.28) (xy 33.02 82.55))
+    (stroke (width 0) (type default))
+  )
+  (wire (pts (xy 45.72 81.28) (xy 45.72 82.55))
+    (stroke (width 0) (type default))
+  )
   (wire (pts (xy 189.23 45.72) (xy 201.93 45.72))
     (stroke (width 0) (type default))
@@
   (wire (pts (xy 143.51 129.54) (xy 148.59 129.54))
     (stroke (width 0) (type solid))
+  )
+  (wire (pts (xy 21.59 88.9) (xy 21.59 90.17))
+    (stroke (width 0) (type default))
   )
   (wire (pts (xy 133.35 132.08) (xy 133.35 133.35))
@@
     (fill (type none))
   )
+  (rectangle (start 17.78 74.93) (end 67.31 97.79)
+    (stroke (width 0) (type dash))
+    (fill (type none))
+  )
   (rectangle (start 182.88 20.32) (end 257.81 78.74)
     (stroke (width 0) (type dash))
@@
     (effects (font (size 1 1)) (justify left bottom))
   )
+  (text "Test points" (at 20.32 73.66 0)
+    (effects (font (size 1.27 1.27)) (justify left bottom))
+  )
   (text "Monitoring" (at 186.1615 18.9286 0)
     (effects (font (size 1.27 1.27)) (justify left bottom))
@@
         (path "/5ad67b7d-c56f-4b00-8953-cc84f90f9708/a004841b-bac3-4d41-b697-5d2e29fa9f3a"
           (reference "#PWR0302") (unit 1)
+        )
+      )
+    )
+  )
+  (symbol (lib_id "Connector:TestPoint") (at 58.42 82.55 180) (unit 1)
+    (in_bom yes) (on_board yes) (dnp no) (fields_autoplaced)
+    (property "Reference" "TP303" (at 60.96 85.217 0)
+      (effects (font (size 1.27 1.27)) (justify right))
+    )
+    (property "Value" "3.3V" (at 60.96 87.757 0)
+      (effects (font (size 1.27 1.27)) (justify right))
+    )
+    (property "Footprint" "TestPoint:TestPoint_Pad_D2.0mm" (at 53.34 82.55 0)
+      (effects (font (size 1.27 1.27)) hide)
+    )
+    (property "Datasheet" "~" (at 53.34 82.55 0)
+      (effects (font (size 1.27 1.27)) hide)
+    )
+    (pin "1")
+    (instances
+      (project "main-board"
+        (path "/5ad67b7d-c56f-4b00-8953-cc84f90f9708/a004841b-bac3-4d41-b697-5d2e29fa9f3a"
+          (reference "TP303") (unit 1)
         )
       )
@@
     )
   )
+  (symbol (lib_id "power:+24V") (at 33.02 81.28 0) (unit 1)
+    (in_bom yes) (on_board yes) (dnp no) (fields_autoplaced)
+    (property "Reference" "#PWR0324" (at 33.02 85.09 0)
+      (effects (font (size 1.27 1.27)) hide)
+    )
+    (property "Value" "+24V" (at 33.02 77.47 0)
+      (effects (font (size 1.27 1.27)))
+    )
+    (property "Footprint" "" (at 33.02 81.28 0)
+      (effects (font (size 1.27 1.27)) hide)
+    )
+    (property "Datasheet" "" (at 33.02 81.28 0)
+      (effects (font (size 1.27 1.27)) hide)
+    )
+    (pin "1")
+    (instances
+      (project "main-board"
+        (path "/5ad67b7d-c56f-4b00-8953-cc84f90f9708/a004841b-bac3-4d41-b697-5d2e29fa9f3a"
+          (reference "#PWR0324") (unit 1)
+        )
+      )
+    )
+  )
   (symbol (lib_id "Device:C_Small") (at 143.51 123.19 0) (unit 1)
     (in_bom yes) (on_board yes) (dnp no)
@@
     )
   )
+  (symbol (lib_id "power:+3.3V") (at 58.42 81.28 0) (unit 1)
+    (in_bom yes) (on_board yes) (dnp no) (fields_autoplaced)
+    (property "Reference" "#PWR0323" (at 58.42 85.09 0)
+      (effects (font (size 1.27 1.27)) hide)
+    )
+    (property "Value" "+3.3V" (at 58.42 77.47 0)
+      (effects (font (size 1.27 1.27)))
+    )
+    (property "Footprint" "" (at 58.42 81.28 0)
+      (effects (font (size 1.27 1.27)) hide)
+    )
+    (property "Datasheet" "" (at 58.42 81.28 0)
+      (effects (font (size 1.27 1.27)) hide)
+    )
+    (pin "1")
+    (instances
+      (project "main-board"
+        (path "/5ad67b7d-c56f-4b00-8953-cc84f90f9708/a004841b-bac3-4d41-b697-5d2e29fa9f3a"
+          (reference "#PWR0323") (unit 1)
+        )
+      )
+    )
+  )
   (symbol (lib_name "GND_1") (lib_id "power:GND") (at 88.9 49.53 0) (unit 1)
     (in_bom yes) (on_board yes) (dnp no)
@@
       (effects (font (size 1.27 1.27)) hide)
     )
-    (property "Value" "GND" (at 88.9 54.61 0)
+    (property "Value" "GND" (at 88.9 53.34 0)
       (effects (font (size 1.27 1.27)))
     )
@@
     )
   )
+  (symbol (lib_id "Connector:TestPoint") (at 45.72 82.55 180) (unit 1)
+    (in_bom yes) (on_board yes) (dnp no) (fields_autoplaced)
+    (property "Reference" "TP302" (at 48.26 85.217 0)
+      (effects (font (size 1.27 1.27)) (justify right))
+    )
+    (property "Value" "5V" (at 48.26 87.757 0)
+      (effects (font (size 1.27 1.27)) (justify right))
+    )
+    (property "Footprint" "TestPoint:TestPoint_Pad_D2.0mm" (at 40.64 82.55 0)
+      (effects (font (size 1.27 1.27)) hide)
+    )
+    (property "Datasheet" "~" (at 40.64 82.55 0)
+      (effects (font (size 1.27 1.27)) hide)
+    )
+    (pin "1")
+    (instances
+      (project "main-board"
+        (path "/5ad67b7d-c56f-4b00-8953-cc84f90f9708/a004841b-bac3-4d41-b697-5d2e29fa9f3a"
+          (reference "TP302") (unit 1)
+        )
+      )
+    )
+  )
   (symbol (lib_name "GND_2") (lib_id "power:GND") (at 193.04 128.27 0) (unit 1)
     (in_bom yes) (on_board yes) (dnp no)
@@
     )
   )
+  (symbol (lib_id "Connector:TestPoint") (at 21.59 88.9 0) (unit 1)
+    (in_bom yes) (on_board yes) (dnp no) (fields_autoplaced)
+    (property "Reference" "TP304" (at 24.13 84.963 0)
+      (effects (font (size 1.27 1.27)) (justify left))
+    )
+    (property "Value" "GND" (at 24.13 87.503 0)
+      (effects (font (size 1.27 1.27)) (justify left))
+    )
+    (property "Footprint" "TestPoint:TestPoint_Pad_D2.0mm" (at 26.67 88.9 0)
+      (effects (font (size 1.27 1.27)) hide)
+    )
+    (property "Datasheet" "~" (at 26.67 88.9 0)
+      (effects (font (size 1.27 1.27)) hide)
+    )
+    (pin "1")
+    (instances
+      (project "main-board"
+        (path "/5ad67b7d-c56f-4b00-8953-cc84f90f9708/a004841b-bac3-4d41-b697-5d2e29fa9f3a"
+          (reference "TP304") (unit 1)
+        )
+      )
+    )
+  )
   (symbol (lib_id "Device:C_Small") (at 101.6 135.89 0) (unit 1)
     (in_bom yes) (on_board yes) (dnp no)
@@
     )
   )
+  (symbol (lib_id "power:+5V") (at 45.72 81.28 0) (unit 1)
+    (in_bom yes) (on_board yes) (dnp no) (fields_autoplaced)
+    (property "Reference" "#PWR0325" (at 45.72 85.09 0)
+      (effects (font (size 1.27 1.27)) hide)
+    )
+    (property "Value" "+5V" (at 45.72 77.47 0)
+      (effects (font (size 1.27 1.27)))
+    )
+    (property "Footprint" "" (at 45.72 81.28 0)
+      (effects (font (size 1.27 1.27)) hide)
+    )
+    (property "Datasheet" "" (at 45.72 81.28 0)
+      (effects (font (size 1.27 1.27)) hide)
+    )
+    (pin "1")
+    (instances
+      (project "main-board"
+        (path "/5ad67b7d-c56f-4b00-8953-cc84f90f9708/a004841b-bac3-4d41-b697-5d2e29fa9f3a"
+          (reference "#PWR0325") (unit 1)
+        )
+      )
+    )
+  )
   (symbol (lib_id "Device:C_Small") (at 160.02 66.04 0) (unit 1)
     (in_bom yes) (on_board yes) (dnp no)
@@
     )
   )
+  (symbol (lib_name "GND_1") (lib_id "power:GND") (at 21.59 90.17 0) (unit 1)
+    (in_bom yes) (on_board yes) (dnp no)
+    (property "Reference" "#PWR0311" (at 21.59 96.52 0)
+      (effects (font (size 1.27 1.27)) hide)
+    )
+    (property "Value" "GND" (at 21.59 93.98 0)
+      (effects (font (size 1.27 1.27)))
+    )
+    (property "Footprint" "" (at 21.59 90.17 0)
+      (effects (font (size 1.27 1.27)) hide)
+    )
+    (property "Datasheet" "" (at 21.59 90.17 0)
+      (effects (font (size 1.27 1.27)) hide)
+    )
+    (pin "1")
+    (instances
+      (project "main-board"
+        (path "/5ad67b7d-c56f-4b00-8953-cc84f90f9708/a004841b-bac3-4d41-b697-5d2e29fa9f3a"
+          (reference "#PWR0311") (unit 1)
+        )
+      )
+    )
+  )
   (symbol (lib_id "Device:C_Small") (at 91.44 135.89 0) (unit 1)
     (in_bom yes) (on_board yes) (dnp no)
@@
         )
       )
+    )
+  )
+  (symbol (lib_id "Connector:TestPoint") (at 33.02 82.55 180) (unit 1)
+    (in_bom yes) (on_board yes) (dnp no) (fields_autoplaced)
+    (property "Reference" "TP301" (at 35.56 85.217 0)
+      (effects (font (size 1.27 1.27)) (justify right))
+    )
+    (property "Value" "24V" (at 35.56 87.757 0)
+      (effects (font (size 1.27 1.27)) (justify right))
+    )
+    (property "Footprint" "TestPoint:TestPoint_Pad_D2.0mm" (at 27.94 82.55 0)
+      (effects (font (size 1.27 1.27)) hide)
+    )
+    (property "Datasheet" "~" (at 27.94 82.55 0)
+      (effects (font (size 1.27 1.27)) hide)
+    )
+    (pin "1")
+    (instances
+      (project "main-board"
+        (path "/5ad67b7d-c56f-4b00-8953-cc84f90f9708/a004841b-bac3-4d41-b697-5d2e29fa9f3a"
+          (reference "TP301") (unit 1)
+        )
+      )

Commit message: Use parts similar to other boards where possible.
Parts:
- C305, C306, C307, C308: MPN GRM21BR71A106KA73L -> GRM21BR61H106KE43L
- C311, C312, C313, C314, C315, C316: value 10uF 35v -> 10uF; MPN GRM21BC8YA106KE11L -> GRM21BR61H106KE43L
Changed lines of the file:
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@@
       (effects (font (size 1.27 1.27)) hide)
     )
-    (property "MPN" "GRM21BR71A106KA73L" (at 193.04 121.92 0)
+    (property "MPN" "GRM21BR61H106KE43L" (at 193.04 121.92 0)
       (effects (font (size 1.27 1.27)) hide)
     )
@@
       (effects (font (size 1.27 1.27)) (justify left))
     )
-    (property "Value" "10uF 35v" (at 111.76 138.43 0)
+    (property "Value" "10uF" (at 111.76 138.43 0)
       (effects (font (size 1.27 1.27)) (justify left))
     )
@@
       (effects (font (size 1.27 1.27)) hide)
     )
-    (property "MPN" "GRM21BC8YA106KE11L " (at 111.76 135.89 0)
+    (property "MPN" "GRM21BR61H106KE43L" (at 111.76 135.89 0)
       (effects (font (size 1.27 1.27)) hide)
     )
@@
       (effects (font (size 1.27 1.27)) hide)
     )
-    (property "MPN" "GRM21BR71A106KA73L" (at 222.25 121.92 0)
+    (property "MPN" "GRM21BR61H106KE43L" (at 222.25 121.92 0)
       (effects (font (size 1.27 1.27)) hide)
     )
@@
       (effects (font (size 1.27 1.27)) hide)
     )
-    (property "MPN" "GRM21BR71A106KA73L" (at 213.36 121.92 0)
+    (property "MPN" "GRM21BR61H106KE43L" (at 213.36 121.92 0)
       (effects (font (size 1.27 1.27)) hide)
     )
@@
       (effects (font (size 1.27 1.27)) (justify left))
     )
-    (property "Value" "10uF 35v" (at 101.6 138.43 0)
+    (property "Value" "10uF" (at 101.6 138.43 0)
       (effects (font (size 1.27 1.27)) (justify left))
     )
@@
       (effects (font (size 1.27 1.27)) hide)
     )
-    (property "MPN" "GRM21BC8YA106KE11L " (at 101.6 135.89 0)
+    (property "MPN" "GRM21BR61H106KE43L" (at 101.6 135.89 0)
       (effects (font (size 1.27 1.27)) hide)
     )
@@
       (effects (font (size 1.27 1.27)) (justify left))
     )
-    (property "Value" "10uF 35v" (at 133.35 138.43 0)
+    (property "Value" "10uF" (at 133.35 138.43 0)
       (effects (font (size 1.27 1.27)) (justify left))
     )
@@
       (effects (font (size 1.27 1.27)) hide)
     )
-    (property "MPN" "GRM21BC8YA106KE11L " (at 133.35 135.89 0)
+    (property "MPN" "GRM21BR61H106KE43L" (at 133.35 135.89 0)
       (effects (font (size 1.27 1.27)) hide)
     )
@@
       (effects (font (size 1.27 1.27)) (justify left))
     )
-    (property "Value" "10uF 35v" (at 121.92 138.43 0)
+    (property "Value" "10uF" (at 121.92 138.43 0)
       (effects (font (size 1.27 1.27)) (justify left))
     )
@@
       (effects (font (size 1.27 1.27)) hide)
     )
-    (property "MPN" "GRM21BC8YA106KE11L " (at 121.92 135.89 0)
+    (property "MPN" "GRM21BR61H106KE43L" (at 121.92 135.89 0)
       (effects (font (size 1.27 1.27)) hide)
     )
@@
       (effects (font (size 1.27 1.27)) (justify left))
     )
-    (property "Value" "10uF 35v" (at 80.01 138.43 0)
+    (property "Value" "10uF" (at 80.01 138.43 0)
       (effects (font (size 1.27 1.27)) (justify left))
     )
@@
       (effects (font (size 1.27 1.27)) hide)
     )
-    (property "MPN" "GRM21BC8YA106KE11L " (at 80.01 135.89 0)
+    (property "MPN" "GRM21BR61H106KE43L" (at 80.01 135.89 0)
       (effects (font (size 1.27 1.27)) hide)
     )
@@
       (effects (font (size 1.27 1.27)) hide)
     )
-    (property "MPN" "GRM21BR71A106KA73L" (at 203.2 121.92 0)
+    (property "MPN" "GRM21BR61H106KE43L" (at 203.2 121.92 0)
       (effects (font (size 1.27 1.27)) hide)
     )
@@
       (effects (font (size 1.27 1.27)) (justify left))
     )
-    (property "Value" "10uF 35v" (at 91.44 138.43 0)
+    (property "Value" "10uF" (at 91.44 138.43 0)
       (effects (font (size 1.27 1.27)) (justify left))
     )
@@
       (effects (font (size 1.27 1.27)) hide)
     )
-    (property "MPN" "GRM21BC8YA106KE11L " (at 91.44 135.89 0)
-      (effects (font (size 1.27 1.27)) hide)
-    )
+    (property "MPN" "GRM21BR61H106KE43L" (at 91.44 135.89 0)
+      (effects (font (size 1.27 1.27)) hide)
+    )
