File: micro.kicad_sch (KiCad schematic)
At the start: 30 parts, among them Q2 BSS138, SW4 SW_Coded_SH-7050, SW5 SW_DIP_x04, SW7 S_D_2, U10 RP2040, U11 W25Q128JVS, U9 74LS151, Y2 12MHz

Commit message: Import the previous main board to match the overall shape, and re-annotate the schematic.
Parts:
- C501: renamed from C54; footprint Capacitor_SMD:C_0402_1005Metric -> Capacitor_SMD:C_0603_1608Metric; MPN (none) -> RM EMK105 B7104KV-F
- C502: renamed from C55; footprint Capacitor_SMD:C_0402_1005Metric -> Capacitor_SMD:C_0603_1608Metric; MPN (none) -> RM EMK105 B7104KV-F
- C503: renamed from C34; footprint Capacitor_SMD:C_0402_1005Metric -> Capacitor_SMD:C_0603_1608Metric; MPN (none) -> RM EMK105 B7104KV-F
- C504: renamed from C48; footprint Capacitor_SMD:C_0402_1005Metric -> Capacitor_SMD:C_0603_1608Metric; MPN (none) -> RM EMK105 B7104KV-F
- C505: renamed from C49; footprint Capacitor_SMD:C_0402_1005Metric -> Capacitor_SMD:C_0603_1608Metric; MPN (none) -> RM EMK105 B7104KV-F
- C506: renamed from C50; footprint Capacitor_SMD:C_0402_1005Metric -> Capacitor_SMD:C_0603_1608Metric; MPN (none) -> RM EMK105 B7104KV-F
- C507: renamed from C51; footprint Capacitor_SMD:C_0402_1005Metric -> Capacitor_SMD:C_0603_1608Metric; MPN (none) -> RM EMK105 B7104KV-F
- C508: renamed from C52; footprint Capacitor_SMD:C_0402_1005Metric -> Capacitor_SMD:C_0603_1608Metric; MPN (none) -> RM EMK105 B7104KV-F
- C509: renamed from C53; footprint Capacitor_SMD:C_0402_1005Metric -> Capacitor_SMD:C_0603_1608Metric; MPN (none) -> RM EMK105 B7104KV-F
- C510: renamed from C56; footprint Capacitor_SMD:C_0402_1005Metric -> Capacitor_SMD:C_0603_1608Metric
- C511: renamed from C36; footprint Capacitor_SMD:C_0402_1005Metric -> Capacitor_SMD:C_0603_1608Metric
- C512: renamed from C32; footprint Capacitor_SMD:C_0402_1005Metric -> Capacitor_SMD:C_0603_1608Metric
- C513: renamed from C33; footprint Capacitor_SMD:C_0402_1005Metric -> Capacitor_SMD:C_0603_1608Metric
- C514: renamed from C35; footprint Capacitor_SMD:C_0402_1005Metric -> Capacitor_SMD:C_0603_1608Metric; MPN (none) -> RM EMK105 B7104KV-F
- R23: footprint Resistor_SMD:R_0402_1005Metric -> Resistor_SMD:R_0603_1608Metric; MPN (none) -> RMCF0603ZT0R00
- R26: value 1k -> 1K; footprint Resistor_SMD:R_0402_1005Metric -> Resistor_SMD:R_0603_1608Metric; MPN RK73H1ETTP1001F -> RC0603FR-101KL
- R502: renamed from R29; value 1k -> 1K; footprint Resistor_SMD:R_0402_1005Metric -> Resistor_SMD:R_0603_1608Metric
- R504: renamed from R28; footprint Resistor_SMD:R_0402_1005Metric -> Resistor_SMD:R_0603_1608Metric
- RN501: renamed from RN2; footprint (none) -> Resistor_SMD:R_Array_Concave_4x0603
- RN502: renamed from RN1; footprint (none) -> Resistor_SMD:R_Array_Concave_4x0603
- SW502: renamed from SW5; footprint (none) -> Button_Switch_SMD:SW_DIP_SPSTx04_Slide_6.7x11.72mm_W6.73mm_P2.54mm_LowProfile_JPin; MPN (none) -> 219-4MST
- renumbered BZ1 to BZ501, SW4 to SW501, SW7 to SW503, U10 to U501, U9 to U502, U11 to U503, Y2 to Y501

Commit message: Finish the draft routing.
Parts:
- removed RN501: 1.8K, Resistor_SMD:R_Array_Concave_4x0603, symbol Device:R_Pack04
- added R505, R506, R507, R508: 1.8K, Resistor_SMD:R_0603_1608Metric, symbol Device:R_Small_US
Connections:
- net +3V3 is gone; now on net +3.3V: C503.1, C504.1, C505.1, C506.1, C507.1, C508.1, C509.1, C511.1, C514.1, R504.1, U501.1 (IOVDD), U501.10 (IOVDD), U501.22 (IOVDD), U501.26 (RUN), U501.33 (IOVDD), U501.42 (IOVDD), U501.43 (ADC_AVDD), U501.44 (VREG_IN), U501.48 (USB_VDD), U501.49 (IOVDD), U503.8 (VCC)
- net +3.3V: now also R505.1, R506.1, R507.1, R508.1
- net DIP_0: now also RN502.4 (R4.1), U502.12 (I7); no longer RN502.1 (R1.1), U502.4 (I0)
- net DIP_1: now also RN502.3 (R3.1), U502.13 (I6); no longer RN502.2 (R2.1), U502.3 (I1)
- net DIP_2: now also RN502.2 (R2.1), U502.14 (I5); no longer RN502.3 (R3.1), U502.2 (I2)
- net DIP_3: now also RN502.1 (R1.1), U502.15 (I4); no longer RN502.4 (R4.1), U502.1 (I3)
- net I2C0_SCL: now also R508.2
- net I2C0_SDA: now also R507.2
- net I2C1_SCL: now also R506.2
- net I2C1_SDA: now also R505.2
- net ID_BIT_0: now also U502.2 (I2); no longer U502.15 (I4)
- net ID_BIT_1: now also U502.3 (I1); no longer U502.14 (I5)
- net ID_BIT_2: now also U502.1 (I3); no longer U502.13 (I6)
- net ID_BIT_3: now also U502.4 (I0); no longer U502.12 (I7)
- net MD_CTRL_STATUS: now also U501.9 (GPIO7); no longer U501.8 (GPIO6)
- net MD_DRV_FAULT: now also U501.8 (GPIO6); no longer U501.9 (GPIO7)
- net MUX_O: now also U501.15 (GPIO12); no longer U501.18 (GPIO15)
- net MUX_S0: now also U501.18 (GPIO15); no longer U501.15 (GPIO12)
- net MUX_S1: now also U501.17 (GPIO14); no longer U501.16 (GPIO13)
- net MUX_S2: now also U501.16 (GPIO13); no longer U501.17 (GPIO14)

Commit message: Improve routings,
Parts:
- added C515: 100nF, Capacitor_SMD:C_0603_1608Metric, symbol Device:C_Small
Connections:
- net +3.3V: now also C515.1
- net GND: now also C515.2
Changed lines of the file:
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@@
+    (stroke (width 0) (type default))
+  )
+  (wire (pts (xy 180.34 139.7) (xy 180.34 140.97))
     (stroke (width 0) (type default))
   )
@@
   )
   (wire (pts (xy 154.94 22.86) (xy 154.94 21.59))
+    (stroke (width 0) (type default))
+  )
+  (wire (pts (xy 180.34 133.35) (xy 180.34 134.62))
     (stroke (width 0) (type default))
   )
@@
     )
   )
+  (symbol (lib_id "power:+3.3V") (at 180.34 133.35 0) (unit 1)
+    (in_bom yes) (on_board yes) (dnp no)
+    (property "Reference" "#PWR059" (at 180.34 137.16 0)
+      (effects (font (size 1.27 1.27)) hide)
+    )
+    (property "Value" "+3.3V" (at 180.34 129.54 0)
+      (effects (font (size 1.27 1.27)))
+    )
+    (property "Footprint" "" (at 180.34 133.35 0)
+      (effects (font (size 1.27 1.27)) hide)
+    )
+    (property "Datasheet" "" (at 180.34 133.35 0)
+      (effects (font (size 1.27 1.27)) hide)
+    )
+    (pin "1")
+    (instances
+      (project "main-board"
+        (path "/5ad67b7d-c56f-4b00-8953-cc84f90f9708/d4025ecd-c2b7-426a-90ae-23d9d1364d9e"
+          (reference "#PWR059") (unit 1)
+        )
+        (path "/5ad67b7d-c56f-4b00-8953-cc84f90f9708/6a867d65-34d4-44e3-a5c9-7709cd333049"
+          (reference "#PWR0406") (unit 1)
+        )
+      )
+    )
+  )
   (symbol (lib_id "Device:R_Small_US") (at 128.27 54.61 270) (unit 1)
     (in_bom yes) (on_board yes) (dnp no)
@@
         (path "/fe216d01-45d7-4b2b-ac5d-8d5d41a286b4"
           (reference "Y1") (unit 1)
+        )
+      )
+    )
+  )
+  (symbol (lib_id "Device:C_Small") (at 180.34 137.16 0) (unit 1)
+    (in_bom yes) (on_board yes) (dnp no)
+    (property "Reference" "C515" (at 183.261 135.9916 0)
+      (effects (font (size 1.27 1.27)) (justify left))
+    )
+    (property "Value" "100nF" (at 183.261 138.303 0)
+      (effects (font (size 1.27 1.27)) (justify left))
+    )
+    (property "Footprint" "Capacitor_SMD:C_0603_1608Metric" (at 180.34 137.16 0)
+      (effects (font (size 1.27 1.27)) hide)
+    )
+    (property "Datasheet" "~" (at 180.34 137.16 0)
+      (effects (font (size 1.27 1.27)) hide)
+    )
+    (property "MPN" "RM EMK105 B7104KV-F" (at 180.34 137.16 0)
+      (effects (font (size 1.27 1.27)) hide)
+    )
+    (pin "1")
+    (pin "2")
+    (instances
+      (project "main-board"
+        (path "/5ad67b7d-c56f-4b00-8953-cc84f90f9708/6a867d65-34d4-44e3-a5c9-7709cd333049"
+          (reference "C515") (unit 1)
+        )
+      )
+      (project "RP2040_minimal"
+        (path "/fe216d01-45d7-4b2b-ac5d-8d5d41a286b4"
+          (reference "C16") (unit 1)
         )
       )
@@
         )
       )
+    )
+  )
+  (symbol (lib_id "power:GND") (at 180.34 140.97 0) (unit 1)
+    (in_bom yes) (on_board yes) (dnp no)
+    (property "Reference" "#PWR0407" (at 180.34 147.32 0)
+      (effects (font (size 1.27 1.27)) hide)
+    )
+    (property "Value" "GND" (at 180.467 145.3642 0)
+      (effects (font (size 1.27 1.27)))
+    )
+    (property "Footprint" "" (at 180.34 140.97 0)
+      (effects (font (size 1.27 1.27)) hide)
+    )
+    (property "Datasheet" "" (at 180.34 140.97 0)
+      (effects (font (size 1.27 1.27)) hide)
+    )
+    (pin "1")
+    (instances
+      (project "main-board"
+        (path "/5ad67b7d-c56f-4b00-8953-cc84f90f9708/6a867d65-34d4-44e3-a5c9-7709cd333049"
+          (reference "#PWR0407") (unit 1)
+        )
+      )
+      (project "RP2040_minimal"
+        (path "/fe216d01-45d7-4b2b-ac5d-8d5d41a286b4"
+          (reference "#PWR023") (unit 1)
+        )
+      )

Commit message: Update MPNs.
Parts:
- C501, C502, C503, C504, C505, C506, C507, C508, C509, C514, C515: MPN RM EMK105 B7104KV-F -> C0603C104K4RAC7081
- C510, C511: MPN (none) -> C0603C105K4RAC7411
- C512, C513: MPN (none) -> 06035C270JAT2A
- Q2: MPN (none) -> BSS138-7-F
- R502: MPN (none) -> RC0603FR-101KL
- R504: MPN (none) -> RC0603JR-1010KL
- R505, R506, R507, R508: MPN (none) -> RC0603FR-101K8L
- RN502: MPN (none) -> CAY16-103J4LF
- SW503: MPN (none) -> TS04-66-65-BK-100-SMT
- U501: MPN (none) -> SC0914(13)
- U503: MPN (none) -> W25Q128JVSIQ
Changed lines of the file:
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@@
+      (effects (font (size 1.27 1.27)) hide)
+    )
+    (property "MPN" "RC0603FR-101K8L" (at 128.27 54.61 0)
       (effects (font (size 1.27 1.27)) hide)
     )
@@
       (effects (font (size 1.27 1.27)) hide)
     )
-    (property "MPN" "RM EMK105 B7104KV-F" (at 180.34 137.16 0)
+    (property "MPN" "C0603C104K4RAC7081" (at 180.34 137.16 0)
       (effects (font (size 1.27 1.27)) hide)
     )
@@
       (effects (font (size 1.27 1.27)) hide)
     )
-    (property "MPN" "RM EMK105 B7104KV-F" (at 143.51 25.4 0)
+    (property "MPN" "C0603C104K4RAC7081" (at 143.51 25.4 0)
       (effects (font (size 1.27 1.27)) hide)
     )
@@
       (effects (font (size 1.27 1.27)) hide)
     )
-    (property "MPN" "RM EMK105 B7104KV-F" (at 86.36 25.4 0)
+    (property "MPN" "C0603C104K4RAC7081" (at 86.36 25.4 0)
       (effects (font (size 1.27 1.27)) hide)
     )
@@
       (effects (font (size 1.27 1.27)) hide)
     )
+    (property "MPN" "RC0603JR-1010KL" (at 40.64 161.29 0)
+      (effects (font (size 1.27 1.27)) hide)
+    )
     (pin "1")
     (pin "2")
@@
     )
     (property "Datasheet" "http://www.winbond.com/resource-files/w25q128jv_dtr%20revc%2003272018%20plus.pdf" (at 68.58 172.72 0)
+      (effects (font (size 1.27 1.27)) hide)
+    )
+    (property "MPN" "W25Q128JVSIQ" (at 68.58 172.72 0)
       (effects (font (size 1.27 1.27)) hide)
     )
@@
       (effects (font (size 1.27 1.27)) hide)
     )
+    (property "MPN" "RC0603FR-101K8L" (at 128.27 46.99 0)
+      (effects (font (size 1.27 1.27)) hide)
+    )
     (pin "1")
     (pin "2")
@@
       (effects (font (size 1.27 1.27)) hide)
     )
-    (property "MPN" "RM EMK105 B7104KV-F" (at 53.34 25.4 0)
+    (property "MPN" "C0603C104K4RAC7081" (at 53.34 25.4 0)
       (effects (font (size 1.27 1.27)) hide)
     )
@@
     )
     (property "Datasheet" "~" (at 128.27 52.07 0)
+      (effects (font (size 1.27 1.27)) hide)
+    )
+    (property "MPN" "RC0603FR-101K8L" (at 128.27 52.07 0)
       (effects (font (size 1.27 1.27)) hide)
     )
@@
       (effects (font (size 1.27 1.27)) hide)
     )
+    (property "MPN" "RC0603FR-101KL" (at 35.56 110.49 0)
+      (effects (font (size 1.27 1.27)) hide)
+    )
     (pin "1")
     (pin "2")
@@
       (effects (font (size 1.27 1.27)) hide)
     )
-    (property "MPN" "RM EMK105 B7104KV-F" (at 86.36 170.18 0)
+    (property "MPN" "C0603C104K4RAC7081" (at 86.36 170.18 0)
       (effects (font (size 1.27 1.27)) hide)
     )
@@
       (effects (font (size 1.27 1.27)) hide)
     )
-    (property "MPN" "RM EMK105 B7104KV-F" (at 120.65 25.4 0)
+    (property "MPN" "C0603C104K4RAC7081" (at 120.65 25.4 0)
       (effects (font (size 1.27 1.27)) hide)
     )
@@
     )
     (property "Datasheet" "~" (at 19.05 110.49 0)
+      (effects (font (size 1.27 1.27)) hide)
+    )
+    (property "MPN" "06035C270JAT2A" (at 19.05 110.49 0)
       (effects (font (size 1.27 1.27)) hide)
     )
@@
     )
     (property "Datasheet" "https://datasheets.raspberrypi.com/rp2040/rp2040-datasheet.pdf" (at 67.31 92.71 0)
+      (effects (font (size 1.27 1.27)) hide)
+    )
+    (property "MPN" "SC0914(13)" (at 67.31 92.71 0)
       (effects (font (size 1.27 1.27)) hide)
     )
@@
       (effects (font (size 1.27 1.27)) hide)
     )
+    (property "MPN" "CAY16-103J4LF" (at 266.7 135.89 0)
+      (effects (font (size 1.27 1.27)) hide)
+    )
     (pin "1")
     (pin "2")
@@
       (effects (font (size 1.27 1.27)) hide)
     )
-    (property "MPN" "RM EMK105 B7104KV-F" (at 109.22 25.4 0)
+    (property "MPN" "C0603C104K4RAC7081" (at 109.22 25.4 0)
       (effects (font (size 1.27 1.27)) hide)
     )
@@
       (effects (font (size 1.27 1.27)) hide)
     )
+    (property "MPN" "RC0603FR-101K8L" (at 128.27 49.53 0)
+      (effects (font (size 1.27 1.27)) hide)
+    )
     (pin "1")
     (pin "2")
@@
       (effects (font (size 1.27 1.27)) (justify left) hide)
     )
+    (property "MPN" "BSS138-7-F" (at 215.9 64.77 0)
+      (effects (font (size 1.27 1.27)) hide)
+    )
     (pin "1")
     (pin "2")
@@
       (effects (font (size 1.27 1.27)) hide)
     )
+    (property "MPN" "06035C270JAT2A" (at 19.05 100.33 0)
+      (effects (font (size 1.27 1.27)) hide)
+    )
     (pin "1")
     (pin "2")
@@
       (effects (font (size 1.27 1.27)) hide)
     )
+    (property "MPN" "TS04-66-65-BK-100-SMT" (at 256.54 154.94 0)
+      (effects (font (size 1.27 1.27)) hide)
+    )
     (pin "1")
     (pin "2")
@@
       (effects (font (size 1.27 1.27)) hide)
     )
-    (property "MPN" "RM EMK105 B7104KV-F" (at 41.91 25.4 0)
+    (property "MPN" "C0603C104K4RAC7081" (at 41.91 25.4 0)
       (effects (font (size 1.27 1.27)) hide)
     )
@@
       (effects (font (size 1.27 1.27)) hide)
     )
-    (property "MPN" "RM EMK105 B7104KV-F" (at 132.08 25.4 0)
+    (property "MPN" "C0603C104K4RAC7081" (at 132.08 25.4 0)
       (effects (font (size 1.27 1.27)) hide)
     )
@@
       (effects (font (size 1.27 1.27)) hide)
     )
+    (property "MPN" "C0603C105K4RAC7411" (at 53.34 38.1 0)
+      (effects (font (size 1.27 1.27)) hide)
+    )
     (pin "1")
     (pin "2")
@@
       (effects (font (size 1.27 1.27)) hide)
     )
-    (property "MPN" "RM EMK105 B7104KV-F" (at 154.94 25.4 0)
+    (property "MPN" "C0603C104K4RAC7081" (at 154.94 25.4 0)
       (effects (font (size 1.27 1.27)) hide)
     )
@@
       (effects (font (size 1.27 1.27)) hide)
     )
-    (property "MPN" "RM EMK105 B7104KV-F" (at 97.79 25.4 0)
+    (property "MPN" "C0603C104K4RAC7081" (at 97.79 25.4 0)
       (effects (font (size 1.27 1.27)) hide)
     )
@@
       (effects (font (size 1.27 1.27)) hide)
     )
+    (property "MPN" "C0603C105K4RAC7411" (at 86.36 38.1 0)
+      (effects (font (size 1.27 1.27)) hide)
+    )
