File: micro.kicad_sch (KiCad schematic)
At the start: 34 parts, among them Q2 BSS138, SW501 SW_Coded_SH-7050, SW502 SW_DIP_x04, SW503 S_D_2, U501 RP2040, U502 74LS151, U503 W25Q128JVS, Y501 12MHz

Commit message: Fix the issues found during testing in schematics.
Parts:
- removed RN502: 10K, Resistor_SMD:R_Array_Concave_4x0603, symbol Device:R_Pack04
- removed U502: 74LS151, Package_SO:SOIC-16_3.9x9.9mm_P1.27mm, symbol 74xx:74LS151
- added C401: 100nF, Capacitor_SMD:C_0603_1608Metric, symbol Device:C_Small
- added D401: WIFI, B2612U:B2612U, symbol B2612U:B2612U
- added D402: MIKONA, B2612U:B2612U, symbol B2612U:B2612U
- added D403: IR / FAULT, B2612U:B2612U, symbol B2612U:B2612U
- added R205 (x6): 1K, Resistor_SMD:R_0603_1608Metric, symbol Device:R_Small_US
- added R401: 10K, Resistor_SMD:R_0603_1608Metric, symbol Device:R_Small_US
- added U502: PI4IOE5V6416, Package_DFN_QFN:WQFN-24-1EP_4x4mm_P0.5mm_EP2.45x2.45mm, symbol PI4IOE5V6416:PI4IOE5V6416
- BZ501: footprint Buzzer_Beeper:MagneticBuzzer_CUI_CMT-8504-100-SMT -> Buzzer_Beeper:Indicator_PUI_AI-1440-TWT-24V-2-R; MPN ST-03BHT -> CPI-137-83T
- R23: value 0 -> 10; MPN RMCF0603ZT0R00 -> RC0603FR-1010RL
- SW501: value SW_Coded_SH-7050 -> SH-7050
- SW502: footprint Button_Switch_SMD:SW_DIP_SPSTx04_Slide_6.7x11.72mm_W6.73mm_P2.54mm_LowProfile_JPin -> Button_Switch_SMD:SW_DIP_SPSTx04_Slide_6.7x11.72mm_W8.61mm_P2.54mm_LowProfile
- SW503: MPN TS04-66-65-BK-100-SMT -> PTS645SL43SMTR92 LFS
Connections:
- net I2C0_SDA is gone; now on net I2C0_SCL: R507.2, U501.6 (GPIO4)
- net +3.3V: now also R401.1, U502.23 (VDD(I2C))
- net +5V: now also C401.1, U502.21 (VDD(P))
- net BUTTON: now also U502.10 (P10); no longer U501.32 (GPIO21)
- net DIP_0: now also SW502.1, U502.8 (P07); no longer SW502.8
- net DIP_1: now also SW502.2, U502.7 (P06); no longer SW502.7
- net DIP_2: now also SW502.3, U502.6 (P05); no longer SW502.6
- net DIP_3: now also SW502.4, U502.5 (P04); no longer SW502.5
- net GND: now also SW502.5, SW502.6, SW502.7, SW502.8, C401.2, R205.1, R205.1, R205.1, R205.1, R205.1, R205.1, U502.18 (ADDR), U502.25 (EPAD), U502.9 (GND); no longer SW502.1, SW502.2, SW502.3, SW502.4
- net I2C0_SCL: now also U502.19 (SCL), U502.20 (SDA)
- net ID_BIT_0: now also U502.3 (P02)
- net ID_BIT_1: now also U502.2 (P01)
- net ID_BIT_2: now also U502.4 (P03)
- net ID_BIT_3: now also U502.1 (P00)
- net UART_RX: now also U501.3 (GPIO1); no longer U501.2 (GPIO0)
- net UART_TX: now also U501.2 (GPIO0); no longer U501.3 (GPIO1)
- net IR renamed CM_INT
- net MUX_O renamed ~{IO_INT}
- net ~{IO_INT}: now also U502.22 (~{INT})
- net MUX_S0: no longer names the net of U501.18 (GPIO15)
- net MUX_S1: no longer names the net of U501.17 (GPIO14)
- net MUX_S2: no longer names the net of U501.16 (GPIO13)
- new net: D401.1 (K1), R205.2
- new net: D401.4 (K2), R205.2
- new net: D403.1 (K1), R205.2
- new net: D403.4 (K2), R205.2
- new net: D402.1 (K1), R205.2
- new net: D402.4 (K2), R205.2
- new net: R401.2, U502.24 (~{RESET})
- new net LED_FAULT: D403.2 (A1), U502.15 (P15)
- new net LED_IR: D403.3 (A2), U502.16 (P16)
- new net LED_MIKONA_CHARGING: D402.2 (A1), U502.13 (P13)
- new net LED_MIKONA_FULL: D402.3 (A2), U502.14 (P14)
- new net LED_SWITCH: U502.17 (P17)
- new net LED_WIFI_ACTIVITY: D401.2 (A1), U502.12 (P12)
- new net LED_WIFI_CONNECTED: D401.3 (A2), U502.11 (P11)
- no-connect marks 3 -> 2
Other:
- note added: "Amber"
- note added: "Blue"
- note added: "Green"
- note added: "IO Expander"
- note added: "LEDs"
- note added: "Orange"
- note added: "Red"
- note added: "Yellow/Green"
- moved on the sheet: BZ501, C515, Q2, R23, SW501, SW502, SW503

Commit message: Applied the fixes to the PCB as well.
Connections:
- net BUTTON: now also U502.5 (P04); no longer U502.10 (P10)
- net DIP_0: now also U502.4 (P03); no longer U502.8 (P07)
- net DIP_1: now also U502.3 (P02); no longer U502.7 (P06)
- net DIP_2: now also U502.2 (P01); no longer U502.6 (P05)
- net DIP_3: now also U502.1 (P00); no longer U502.5 (P04)
- net I2C0_SCL: no longer R507.2, U501.6 (GPIO4), U502.20 (SDA)
- net ID_BIT_0: now also U502.15 (P15); no longer U502.3 (P02)
- net ID_BIT_1: now also U502.17 (P17); no longer U502.2 (P01)
- net ID_BIT_2: now also U502.14 (P14); no longer U502.4 (P03)
- net ID_BIT_3: now also U502.16 (P16); no longer U502.1 (P00)
- net LED_FAULT: now also U502.6 (P05); no longer U502.15 (P15)
- net LED_IR: now also U502.7 (P06); no longer U502.16 (P16)
- net LED_MIKONA_CHARGING: now also U502.8 (P07); no longer U502.13 (P13)
- net LED_MIKONA_FULL: now also U502.10 (P10); no longer U502.14 (P14)
- net LED_SWITCH: now also U502.13 (P13); no longer U502.17 (P17)
- net LED_WIFI_ACTIVITY: now also U502.11 (P11); no longer U502.12 (P12)
- net LED_WIFI_CONNECTED: now also U502.12 (P12); no longer U502.11 (P11)
- new net I2C0_SDA: R507.2, U501.6 (GPIO4), U502.20 (SDA)
- no-connect marks 2 -> 6

Commit message: Change on-board LEDs to vertical diffuse.
Parts:
- D2: MPN SML-A12M8TT86N -> B1911PG--20D000514U1930
Changed lines of the file:
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@@
       (effects (font (size 1.27 1.27)) hide)
     )
-    (property "MPN" "SML-A12M8TT86N" (at 139.7 118.11 0)
+    (property "MPN" "B1911PG--20D000514U1930" (at 139.7 118.11 0)
       (effects (font (size 1.27 1.27)) hide)
     )
