File: motors.kicad_sch (KiCad schematic)
At the start: 15 parts, among them J705 ENC1, J706 ENC2, J707 M1, J708 M2, J711 ENC3, J712 ENC4, J713 M3, J714 M4, J717 ENCD, J718 MD

Commit message: Improve routings,
Parts:
- J705, J706, J711, J712, J717: symbol Connector_Generic_MountingPin:Conn_01x06_MountingPin -> Connector_Generic:Conn_01x06
Connections:
- net GND: no longer J705.MP (MountPin), J706.MP (MountPin), J711.MP (MountPin), J712.MP (MountPin), J717.MP (MountPin)
Changed lines of the file:
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@@
     (stroke (width 0) (type default))
   )
-  (wire (pts (xy 204.47 86.36) (xy 204.47 87.63))
-    (stroke (width 0) (type default))
-  )
   (wire (pts (xy 106.68 68.58) (xy 107.95 68.58))
     (stroke (width 0) (type default))
@@
     (stroke (width 0) (type default))
   )
-  (wire (pts (xy 262.89 86.36) (xy 262.89 87.63))
-    (stroke (width 0) (type default))
-  )
   (wire (pts (xy 163.83 120.65) (xy 175.26 120.65))
     (stroke (width 0) (type default))
@@
     (stroke (width 0) (type default))
   )
-  (wire (pts (xy 204.47 154.94) (xy 204.47 156.21))
-    (stroke (width 0) (type default))
-  )
   (wire (pts (xy 106.68 26.67) (xy 107.95 26.67))
     (stroke (width 0) (type default))
@@
     (stroke (width 0) (type default))
   )
-  (wire (pts (xy 262.89 120.65) (xy 262.89 121.92))
-    (stroke (width 0) (type default))
-  )
   (wire (pts (xy 95.25 41.91) (xy 106.68 41.91))
     (stroke (width 0) (type default))
@@
     (stroke (width 0) (type default))
   )
-  (wire (pts (xy 204.47 120.65) (xy 204.47 121.92))
-    (stroke (width 0) (type default))
-  )
   (wire (pts (xy 73.66 78.74) (xy 74.93 78.74))
     (stroke (width 0) (type default))
@@
     )
   )
-  (symbol (lib_id "Connector_Generic_MountingPin:Conn_01x06_MountingPin") (at 262.89 107.95 0) (unit 1)
+  (symbol (lib_id "Connector_Generic:Conn_01x06") (at 262.89 107.95 0) (unit 1)
     (in_bom yes) (on_board yes) (dnp no)
     (property "Reference" "J712" (at 261.62 100.33 0)
@@
     (pin "5")
     (pin "6")
-    (pin "MP")
     (instances
       (project "main-board"
@@
     )
   )
-  (symbol (lib_id "Connector_Generic_MountingPin:Conn_01x06_MountingPin") (at 204.47 73.66 0) (unit 1)
+  (symbol (lib_id "Connector_Generic:Conn_01x06") (at 204.47 73.66 0) (unit 1)
     (in_bom yes) (on_board yes) (dnp no)
     (property "Reference" "J705" (at 203.2 66.04 0)
@@
     (pin "5")
     (pin "6")
-    (pin "MP")
     (instances
       (project "main-board"
@@
     )
   )
-  (symbol (lib_id "Connector_Generic_MountingPin:Conn_01x06_MountingPin") (at 204.47 142.24 0) (unit 1)
+  (symbol (lib_id "Connector_Generic:Conn_01x06") (at 204.47 142.24 0) (unit 1)
     (in_bom yes) (on_board yes) (dnp yes)
     (property "Reference" "J717" (at 203.2 134.62 0)
@@
     (pin "5")
     (pin "6")
-    (pin "MP")
     (instances
       (project "main-board"
@@
     )
   )
-  (symbol (lib_id "Connector_Generic_MountingPin:Conn_01x06_MountingPin") (at 204.47 107.95 0) (unit 1)
+  (symbol (lib_id "Connector_Generic:Conn_01x06") (at 204.47 107.95 0) (unit 1)
     (in_bom yes) (on_board yes) (dnp no)
     (property "Reference" "J711" (at 203.2 100.33 0)
@@
     (pin "5")
     (pin "6")
-    (pin "MP")
     (instances
       (project "main-board"
@@
     )
   )
-  (symbol (lib_id "power:GND") (at 204.47 156.21 0) (unit 1)
-    (in_bom yes) (on_board yes) (dnp no)
-    (property "Reference" "#PWR030" (at 204.47 162.56 0)
-      (effects (font (size 1.27 1.27)) hide)
-    )
-    (property "Value" "GND" (at 207.01 160.02 0)
-      (effects (font (size 1.27 1.27)) (justify right))
-    )
-    (property "Footprint" "" (at 204.47 156.21 0)
-      (effects (font (size 1.27 1.27)) hide)
-    )
-    (property "Datasheet" "" (at 204.47 156.21 0)
-      (effects (font (size 1.27 1.27)) hide)
-    )
-    (pin "1")
-    (instances
-      (project "motor-driver"
-        (path "/314549f2-cc46-4559-991a-ae9411f3d209/25794513-4b05-4cf2-b97c-a9dcfa280e83"
-          (reference "#PWR030") (unit 1)
-        )
-        (path "/314549f2-cc46-4559-991a-ae9411f3d209"
-          (reference "#PWR074") (unit 1)
-        )
-      )
-      (project "main-board"
-        (path "/5ad67b7d-c56f-4b00-8953-cc84f90f9708/cf228cb6-f574-4df0-9eba-d154373551fd"
-          (reference "#PWR0748") (unit 1)
-        )
-      )
-    )
-  )
   (symbol (lib_id "Connector_Generic:Conn_01x08") (at 180.34 110.49 0) (unit 1)
     (in_bom yes) (on_board yes) (dnp no)
@@
     )
   )
-  (symbol (lib_id "power:GND") (at 262.89 87.63 0) (unit 1)
-    (in_bom yes) (on_board yes) (dnp no)
-    (property "Reference" "#PWR030" (at 262.89 93.98 0)
-      (effects (font (size 1.27 1.27)) hide)
-    )
-    (property "Value" "GND" (at 265.43 91.44 0)
-      (effects (font (size 1.27 1.27)) (justify right))
-    )
-    (property "Footprint" "" (at 262.89 87.63 0)
-      (effects (font (size 1.27 1.27)) hide)
-    )
-    (property "Datasheet" "" (at 262.89 87.63 0)
-      (effects (font (size 1.27 1.27)) hide)
-    )
-    (pin "1")
-    (instances
-      (project "motor-driver"
-        (path "/314549f2-cc46-4559-991a-ae9411f3d209/25794513-4b05-4cf2-b97c-a9dcfa280e83"
-          (reference "#PWR030") (unit 1)
-        )
-        (path "/314549f2-cc46-4559-991a-ae9411f3d209"
-          (reference "#PWR074") (unit 1)
-        )
-      )
-      (project "main-board"
-        (path "/5ad67b7d-c56f-4b00-8953-cc84f90f9708/cf228cb6-f574-4df0-9eba-d154373551fd"
-          (reference "#PWR0724") (unit 1)
-        )
-      )
-    )
-  )
   (symbol (lib_id "Immortals:MotorDriver") (at 49.53 36.83 0) (unit 1)
     (in_bom yes) (on_board yes) (dnp no)
@@
     )
   )
-  (symbol (lib_id "Connector_Generic_MountingPin:Conn_01x06_MountingPin") (at 262.89 73.66 0) (unit 1)
+  (symbol (lib_id "Connector_Generic:Conn_01x06") (at 262.89 73.66 0) (unit 1)
     (in_bom yes) (on_board yes) (dnp no)
     (property "Reference" "J706" (at 261.62 66.04 0)
@@
     (pin "5")
     (pin "6")
-    (pin "MP")
     (instances
       (project "main-board"
@@
     )
   )
-  (symbol (lib_id "power:GND") (at 204.47 121.92 0) (unit 1)
-    (in_bom yes) (on_board yes) (dnp no)
-    (property "Reference" "#PWR030" (at 204.47 128.27 0)
-      (effects (font (size 1.27 1.27)) hide)
-    )
-    (property "Value" "GND" (at 207.01 125.73 0)
-      (effects (font (size 1.27 1.27)) (justify right))
-    )
-    (property "Footprint" "" (at 204.47 121.92 0)
-      (effects (font (size 1.27 1.27)) hide)
-    )
-    (property "Datasheet" "" (at 204.47 121.92 0)
-      (effects (font (size 1.27 1.27)) hide)
-    )
-    (pin "1")
-    (instances
-      (project "motor-driver"
-        (path "/314549f2-cc46-4559-991a-ae9411f3d209/25794513-4b05-4cf2-b97c-a9dcfa280e83"
-          (reference "#PWR030") (unit 1)
-        )
-        (path "/314549f2-cc46-4559-991a-ae9411f3d209"
-          (reference "#PWR074") (unit 1)
-        )
-      )
-      (project "main-board"
-        (path "/5ad67b7d-c56f-4b00-8953-cc84f90f9708/cf228cb6-f574-4df0-9eba-d154373551fd"
-          (reference "#PWR0738") (unit 1)
-        )
-      )
-    )
-  )
   (symbol (lib_id "power:+24V") (at 104.14 26.67 0) (unit 1)
     (in_bom yes) (on_board yes) (dnp no)
@@
     )
   )
-  (symbol (lib_id "power:GND") (at 204.47 87.63 0) (unit 1)
-    (in_bom yes) (on_board yes) (dnp no)
-    (property "Reference" "#PWR030" (at 204.47 93.98 0)
-      (effects (font (size 1.27 1.27)) hide)
-    )
-    (property "Value" "GND" (at 207.01 91.44 0)
-      (effects (font (size 1.27 1.27)) (justify right))
-    )
-    (property "Footprint" "" (at 204.47 87.63 0)
-      (effects (font (size 1.27 1.27)) hide)
-    )
-    (property "Datasheet" "" (at 204.47 87.63 0)
-      (effects (font (size 1.27 1.27)) hide)
-    )
-    (pin "1")
-    (instances
-      (project "motor-driver"
-        (path "/314549f2-cc46-4559-991a-ae9411f3d209/25794513-4b05-4cf2-b97c-a9dcfa280e83"
-          (reference "#PWR030") (unit 1)
-        )
-        (path "/314549f2-cc46-4559-991a-ae9411f3d209"
-          (reference "#PWR074") (unit 1)
-        )
-      )
-      (project "main-board"
-        (path "/5ad67b7d-c56f-4b00-8953-cc84f90f9708/cf228cb6-f574-4df0-9eba-d154373551fd"
-          (reference "#PWR0723") (unit 1)
-        )
-      )
-    )
-  )
   (symbol (lib_id "power:+5V") (at 224.79 113.03 90) (unit 1)
     (in_bom yes) (on_board yes) (dnp no)
@@
         )
       )
-    )
-  )
-  (symbol (lib_id "power:GND") (at 262.89 121.92 0) (unit 1)
-    (in_bom yes) (on_board yes) (dnp no)
-    (property "Reference" "#PWR030" (at 262.89 128.27 0)
-      (effects (font (size 1.27 1.27)) hide)
-    )
-    (property "Value" "GND" (at 265.43 125.73 0)
-      (effects (font (size 1.27 1.27)) (justify right))
-    )
-    (property "Footprint" "" (at 262.89 121.92 0)
-      (effects (font (size 1.27 1.27)) hide)
-    )
-    (property "Datasheet" "" (at 262.89 121.92 0)
-      (effects (font (size 1.27 1.27)) hide)
-    )
-    (pin "1")
-    (instances
-      (project "motor-driver"
-        (path "/314549f2-cc46-4559-991a-ae9411f3d209/25794513-4b05-4cf2-b97c-a9dcfa280e83"
-          (reference "#PWR030") (unit 1)
-        )
-        (path "/314549f2-cc46-4559-991a-ae9411f3d209"
-          (reference "#PWR074") (unit 1)
-        )
-      )
-      (project "main-board"
-        (path "/5ad67b7d-c56f-4b00-8953-cc84f90f9708/cf228cb6-f574-4df0-9eba-d154373551fd"
-          (reference "#PWR0739") (unit 1)
-        )
-      )

Commit message: Update MPNs.
Parts:
- J705, J706, J711, J712, J717: MPN (none) -> 0532610671
Changed lines of the file:
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@@
+      (effects (font (size 1.27 1.27)) hide)
+    )
+    (property "MPN" "0532610671" (at 262.89 107.95 0)
       (effects (font (size 1.27 1.27)) hide)
     )
@@
       (effects (font (size 1.27 1.27)) hide)
     )
+    (property "MPN" "0532610671" (at 204.47 73.66 0)
+      (effects (font (size 1.27 1.27)) hide)
+    )
     (pin "1")
     (pin "2")
@@
     )
     (property "Datasheet" "~" (at 204.47 142.24 0)
+      (effects (font (size 1.27 1.27)) hide)
+    )
+    (property "MPN" "0532610671" (at 204.47 142.24 0)
       (effects (font (size 1.27 1.27)) hide)
     )
@@
       (effects (font (size 1.27 1.27)) hide)
     )
+    (property "MPN" "0532610671" (at 204.47 107.95 0)
+      (effects (font (size 1.27 1.27)) hide)
+    )
     (pin "1")
     (pin "2")
@@
       (effects (font (size 1.27 1.27)) hide)
     )
+    (property "MPN" "0532610671" (at 262.89 73.66 0)
+      (effects (font (size 1.27 1.27)) hide)
+    )

Commit message: Add MPNs for CM4 and motor drivers.
Parts:
- U1, U2, U3, U4, U5: MPN (none) -> 61032021821 + NPPC101KFXC-RC
Changed lines of the file:
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@@
+      (effects (font (size 1.27 1.27)) hide)
+    )
+    (property "MPN" "61032021821 + NPPC101KFXC-RC" (at 49.53 162.56 0)
       (effects (font (size 1.27 1.27)) hide)
     )
@@
       (effects (font (size 1.27 1.27)) hide)
     )
+    (property "MPN" "61032021821 + NPPC101KFXC-RC" (at 146.05 36.83 0)
+      (effects (font (size 1.27 1.27)) hide)
+    )
     (pin "1")
     (pin "10")
@@
       (effects (font (size 1.27 1.27)) hide)
     )
+    (property "MPN" "61032021821 + NPPC101KFXC-RC" (at 114.3 78.74 0)
+      (effects (font (size 1.27 1.27)) hide)
+    )
     (pin "1")
     (pin "10")
@@
       (effects (font (size 1.27 1.27)) hide)
     )
+    (property "MPN" "61032021821 + NPPC101KFXC-RC" (at 49.53 120.65 0)
+      (effects (font (size 1.27 1.27)) hide)
+    )
     (pin "1")
     (pin "10")
@@
       (effects (font (size 1.27 1.27)) hide)
     )
+    (property "MPN" "61032021821 + NPPC101KFXC-RC" (at 49.53 36.83 0)
+      (effects (font (size 1.27 1.27)) hide)
+    )
     (pin "1")
     (pin "10")
@@
       (effects (font (size 1.27 1.27)) hide)
     )
+    (property "MPN" "61032021821 + NPPC101KFXC-RC" (at 114.3 36.83 0)
+      (effects (font (size 1.27 1.27)) hide)
+    )
     (pin "1")
     (pin "10")
@@
       (effects (font (size 1.27 1.27)) hide)
     )
+    (property "MPN" "61032021821 + NPPC101KFXC-RC" (at 114.3 162.56 0)
+      (effects (font (size 1.27 1.27)) hide)
+    )
     (pin "1")
     (pin "10")
@@
       (effects (font (size 1.27 1.27)) hide)
     )
+    (property "MPN" "61032021821 + NPPC101KFXC-RC" (at 114.3 120.65 0)
+      (effects (font (size 1.27 1.27)) hide)
+    )
     (pin "1")
     (pin "10")
@@
       (effects (font (size 1.27 1.27)) hide)
     )
+    (property "MPN" "61032021821 + NPPC101KFXC-RC" (at 49.53 78.74 0)
+      (effects (font (size 1.27 1.27)) hide)
+    )
     (pin "1")
     (pin "10")
@@
       (effects (font (size 1.27 1.27)) hide)
     )
+    (property "MPN" "61032021821 + NPPC101KFXC-RC" (at 210.82 36.83 0)
+      (effects (font (size 1.27 1.27)) hide)
+    )

Commit message: Fix the issues found during testing in schematics.
Connections:
- net +3.3V: now also U1.1 (3.3V), U2.1 (3.3V), U3.1 (3.3V), U4.1 (3.3V), U5.1 (3.3V); no longer U1.3 (3.3V), U2.3 (3.3V), U3.3 (3.3V), U4.3 (3.3V), U5.3 (3.3V)
- net +5V: now also U1.3 (5V), U2.3 (5V), U3.3 (5V), U4.3 (5V), U5.3 (5V); no longer U1.1 (5V), U2.1 (5V), U3.1 (5V), U4.1 (5V), U5.1 (5V)
- net GND: now also U1.14 (GND), U2.14 (GND), U3.14 (GND), U4.14 (GND), U5.14 (GND)
- net M1_ENC_A: now also U1.2 (ENC_A); no longer U1.4 (ENC_A)
- net M1_ENC_B: now also U1.4 (ENC_B); no longer U1.6 (ENC_B)
- net M1_ENC_C: now also U1.6 (ENC_C); no longer U1.8 (ENC_C)
- net M1_HALL_UX: now also U1.8 (HALL_UX); no longer U1.10 (HALL_UX)
- net M1_HALL_V: now also U1.10 (HALL_V); no longer U1.12 (HALL_V)
- net M1_HALL_WY: now also U1.12 (HALL_WY); no longer U1.14 (HALL_WY)
- net M2_ENC_A: now also U2.2 (ENC_A); no longer U2.4 (ENC_A)
- net M2_ENC_B: now also U2.4 (ENC_B); no longer U2.6 (ENC_B)
- net M2_ENC_C: now also U2.6 (ENC_C); no longer U2.8 (ENC_C)
- net M2_HALL_UX: now also U2.8 (HALL_UX); no longer U2.10 (HALL_UX)
- net M2_HALL_V: now also U2.10 (HALL_V); no longer U2.12 (HALL_V)
- net M2_HALL_WY: now also U2.12 (HALL_WY); no longer U2.14 (HALL_WY)
- net M3_ENC_A: now also U3.2 (ENC_A); no longer U3.4 (ENC_A)
- net M3_ENC_B: now also U3.4 (ENC_B); no longer U3.6 (ENC_B)
- net M3_ENC_C: now also U3.6 (ENC_C); no longer U3.8 (ENC_C)
- net M3_HALL_UX: now also U3.8 (HALL_UX); no longer U3.10 (HALL_UX)
- net M3_HALL_V: now also U3.10 (HALL_V); no longer U3.12 (HALL_V)
- net M3_HALL_WY: now also U3.12 (HALL_WY); no longer U3.14 (HALL_WY)
- net M4_ENC_A: now also U4.2 (ENC_A); no longer U4.4 (ENC_A)
- net M4_ENC_B: now also U4.4 (ENC_B); no longer U4.6 (ENC_B)
- net M4_ENC_C: now also U4.6 (ENC_C); no longer U4.8 (ENC_C)
- net M4_HALL_UX: now also U4.8 (HALL_UX); no longer U4.10 (HALL_UX)
- net M4_HALL_V: now also U4.10 (HALL_V); no longer U4.12 (HALL_V)
- net M4_HALL_WY: now also U4.12 (HALL_WY); no longer U4.14 (HALL_WY)
- net MD_ENC_A: now also U5.2 (ENC_A); no longer U5.4 (ENC_A)
- net MD_ENC_B: now also U5.4 (ENC_B); no longer U5.6 (ENC_B)
- net MD_ENC_C: now also U5.6 (ENC_C); no longer U5.8 (ENC_C)
- net MD_HALL_UX: now also U5.8 (HALL_UX); no longer U5.10 (HALL_UX)
- net MD_HALL_V: now also U5.10 (HALL_V); no longer U5.12 (HALL_V)
- net MD_HALL_WY: now also U5.12 (HALL_WY); no longer U5.14 (HALL_WY)
