File: sensors.kicad_sch (KiCad schematic)
At the start: 11 parts, among them J24 Qwiic, J602 IR, Q601 BSS138, U601 ICM-42688-P

Commit message: Update MPNs.
Parts:
- C601, C602: MPN RM EMK105 B7104KV-F -> C0603C104K4RAC7081
- C603: MPN (none) -> CL21B225KOFNNNE
- C604: MPN (none) -> C0603C103M5RAC7411
- Q601: MPN (none) -> BSS138-7-F
- R601: MPN (none) -> RC0603JR-07300RL
- R602: MPN (none) -> RC0603FR-0736RL
- U601: MPN (none) -> ICM-42688-P
Changed lines of the file:
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@@
+      (effects (font (size 1.27 1.27)) hide)
+    )
+    (property "MPN" "RC0603FR-0736RL" (at 217.17 76.2 0)
       (effects (font (size 1.27 1.27)) hide)
     )
@@
     )
     (property "Datasheet" "~" (at 241.3 137.16 0)
+      (effects (font (size 1.27 1.27)) hide)
+    )
+    (property "MPN" "C0603C103M5RAC7411" (at 241.3 137.16 0)
       (effects (font (size 1.27 1.27)) hide)
     )
@@
       (effects (font (size 1.27 1.27)) (justify left) hide)
     )
+    (property "MPN" "BSS138-7-F" (at 200.66 81.28 0)
+      (effects (font (size 1.27 1.27)) hide)
+    )
     (pin "1")
     (pin "2")
@@
       (effects (font (size 1.27 1.27)) hide)
     )
-    (property "MPN" "RM EMK105 B7104KV-F" (at 241.3 116.84 0)
+    (property "MPN" "C0603C104K4RAC7081" (at 241.3 116.84 0)
       (effects (font (size 1.27 1.27)) hide)
     )
@@
       (effects (font (size 1.27 1.27)) hide)
     )
-    (property "MPN" "RM EMK105 B7104KV-F" (at 193.04 68.58 0)
+    (property "MPN" "C0603C104K4RAC7081" (at 193.04 68.58 0)
       (effects (font (size 1.27 1.27)) hide)
     )
@@
     )
     (property "Datasheet" "~" (at 227.33 71.12 0)
+      (effects (font (size 1.27 1.27)) hide)
+    )
+    (property "MPN" "RC0603JR-07300RL" (at 227.33 71.12 0)
       (effects (font (size 1.27 1.27)) hide)
     )
@@
       (effects (font (size 1.27 1.27)) hide)
     )
+    (property "MPN" "CL21B225KOFNNNE" (at 251.46 116.84 0)
+      (effects (font (size 1.27 1.27)) hide)
+    )
     (pin "1")
     (pin "2")
@@
       (effects (font (size 1.27 1.27)) hide)
     )
+    (property "MPN" "ICM-42688-P" (at 200.66 127 0)
+      (effects (font (size 1.27 1.27)) hide)
+    )

Commit message: Fix the issues found during testing in schematics.
Parts:
- J602: footprint Connector_JST:JST_SH_SM04B-SRSS-TB_1x04-1MP_P1.00mm_Horizontal -> XH-SM4:CONN_S4B-XH-SM4-TB_JST
- R603: value 0 -> 10; MPN RMCF0603ZT0R00 -> RC0603FR-1010RL
Changed lines of the file:
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@@
       (effects (font (size 1.27 1.27)) (justify left))
     )
-    (property "Footprint" "Connector_JST:JST_SH_SM04B-SRSS-TB_1x04-1MP_P1.00mm_Horizontal" (at 237.49 73.66 0)
+    (property "Footprint" "XH-SM4:CONN_S4B-XH-SM4-TB_JST" (at 237.49 73.66 0)
       (effects (font (size 1.27 1.27)) hide)
     )
@@
       (effects (font (size 1.27 1.27)))
     )
-    (property "Value" "0" (at 193.04 80.01 90)
+    (property "Value" "10" (at 193.04 80.01 90)
       (effects (font (size 1.27 1.27)))
     )
@@
       (effects (font (size 1.27 1.27)) hide)
     )
-    (property "MPN" "RMCF0603ZT0R00" (at 190.5 81.28 0)
+    (property "MPN" "RC0603FR-1010RL" (at 190.5 81.28 0)
       (effects (font (size 1.27 1.27)) hide)
     )

Commit message: Use parts similar to other boards where possible.
Parts:
- C603: MPN CL21B225KOFNNNE -> CC0805KKX7R9BB225
Changed lines of the file:
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@@
       (effects (font (size 1.27 1.27)) hide)
     )
-    (property "MPN" "CL21B225KOFNNNE" (at 251.46 116.84 0)
+    (property "MPN" "CC0805KKX7R9BB225" (at 251.46 116.84 0)
       (effects (font (size 1.27 1.27)) hide)
     )

Commit message: Fix the 24v sense res and the IR port MPN.
Parts:
- J602: MPN SM04B-SRSS-TB(LF)(SN) -> S4B-XH-SM4-TB(LF)(SN)
Changed lines of the file:
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@@
       (effects (font (size 1.27 1.27)) hide)
     )
-    (property "MPN" "SM04B-SRSS-TB(LF)(SN)" (at 237.49 73.66 0)
+    (property "MPN" "S4B-XH-SM4-TB(LF)(SN)" (at 237.49 73.66 0)
       (effects (font (size 1.27 1.27)) hide)
     )
